File: PCB/BerthaBluetooth/v1/v1.sch (EAGLE design)
At the start: 112 parts, among them CON1 SPI, IC1 REG1117, J1 RJ12, J2 RJ12, J3 RJ12, J4 RJ12, J5 RJ12, J6 RJ12, Q1 BSP613P, Q10 BSP613P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

Commit message: Update labels
Parts:
- Q1, Q10, Q2, Q3, Q4, Q5, Q6, Q8, Q9: value BSP613P -> BSP75
- R25, R33, R5: value RJ12 -> 1k
- X4: value MINI-USB-SCHIELD-32005-201 -> MINI-USB
Changed lines of the file:
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@@
 <part name="P+8" library="supply1" deviceset="+12V" device=""/>
 <part name="LED2" library="lpatiny" deviceset="LED3MM" device="" value="Blue"/>
-<part name="R25" library="rcl" deviceset="R-EU_" device="R0805" value="RJ12"/>
+<part name="R25" library="rcl" deviceset="R-EU_" device="R0805" value="1k"/>
 <part name="LED3" library="adafruit" deviceset="LED" device="CHIP-LED0805" value="RED"/>
 <part name="R27" library="rcl" deviceset="R-EU_" device="R0805" value="1K"/>
@@
 <part name="GND22" library="supply1" deviceset="GND" device=""/>
 <part name="SUPPLY7" library="supply1" deviceset="+5V" device=""/>
-<part name="R33" library="rcl" deviceset="R-EU_" device="R0805" value="RJ12"/>
+<part name="R33" library="rcl" deviceset="R-EU_" device="R0805" value="1k"/>
 <part name="P+13" library="supply1" deviceset="+12V" device=""/>
 <part name="LED6" library="lpatiny" deviceset="LED3MM" device="" value="Blue"/>
-<part name="R5" library="rcl" deviceset="R-EU_" device="R0805" value="RJ12"/>
+<part name="R5" library="rcl" deviceset="R-EU_" device="R0805" value="1k"/>
 <part name="J4" library="lpatiny" deviceset="RJ12" device="STRAIGHT" value="RJ12"/>
 <part name="GND23" library="supply1" deviceset="GND" device=""/>
@@
 <part name="RL7" library="rcl" deviceset="R-EU_" device="R0805" value="1K"/>
 <part name="GND1" library="supply1" deviceset="GND" device=""/>
-<part name="Q1" library="infineon" deviceset="BSP613P" device=""/>
-<part name="Q2" library="infineon" deviceset="BSP613P" device=""/>
-<part name="Q4" library="infineon" deviceset="BSP613P" device=""/>
-<part name="Q5" library="infineon" deviceset="BSP613P" device=""/>
-<part name="Q6" library="infineon" deviceset="BSP613P" device=""/>
+<part name="Q1" library="infineon" deviceset="BSP613P" device="" value="BSP75"/>
+<part name="Q2" library="infineon" deviceset="BSP613P" device="" value="BSP75"/>
+<part name="Q4" library="infineon" deviceset="BSP613P" device="" value="BSP75"/>
+<part name="Q5" library="infineon" deviceset="BSP613P" device="" value="BSP75"/>
+<part name="Q6" library="infineon" deviceset="BSP613P" device="" value="BSP75"/>
 <part name="GND29" library="supply1" deviceset="GND" device=""/>
 <part name="+5VA2" library="supply1" deviceset="+5V" device=""/>
@@
 <part name="SUPPLY4" library="supply2" deviceset="+5V/1" device=""/>
 <part name="P+11" library="supply1" deviceset="+5V" device=""/>
-<part name="X4" library="con-cypressindustries" deviceset="MINI-USB-SCHIELD-" device="32005-201"/>
+<part name="X4" library="con-cypressindustries" deviceset="MINI-USB-SCHIELD-" device="32005-201" value="MINI-USB"/>
 <part name="R24" library="resistor" deviceset="R-EU_" device="M1206" value="22"/>
 <part name="R31" library="resistor" deviceset="R-EU_" device="M1206" value="22"/>
@@
 <part name="LED1" library="lpatiny" deviceset="LED3MM" device="" value="Blue"/>
 <part name="R20" library="rcl" deviceset="R-EU_" device="R0805" value="1k"/>
-<part name="Q3" library="infineon" deviceset="BSP613P" device=""/>
+<part name="Q3" library="infineon" deviceset="BSP613P" device="" value="BSP75"/>
 <part name="GND26" library="supply1" deviceset="GND" device=""/>
 <part name="RGB-J1" library="lpatiny" deviceset="RJ12" device="STRAIGHT-RGB" value="RJ12"/>
@@
 <part name="P+41" library="supply1" deviceset="+5V" device=""/>
 <part name="P+42" library="supply1" deviceset="+12V" device=""/>
-<part name="Q8" library="infineon" deviceset="BSP613P" device=""/>
-<part name="Q9" library="infineon" deviceset="BSP613P" device=""/>
-<part name="Q10" library="infineon" deviceset="BSP613P" device=""/>
+<part name="Q8" library="infineon" deviceset="BSP613P" device="" value="BSP75"/>
+<part name="Q9" library="infineon" deviceset="BSP613P" device="" value="BSP75"/>
+<part name="Q10" library="infineon" deviceset="BSP613P" device="" value="BSP75"/>
 <part name="GND33" library="supply1" deviceset="GND" device=""/>
 <part name="GND34" library="supply1" deviceset="GND" device=""/>
