File: PCB/Linear Sensor/v1.1/linearSensor.brd (EAGLE design)
At the start: 63.5 x 35.8 mm, 43 parts, among them CON1 SPI, IC1 REG1117, Q1 BSP613P, X3 16MHz, X4 MINI-USB

Commit message: Create new verison
Parts:
- Q1: value BSP613P -> BSP75
Changed lines of the file:
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@@
 <layer number="19" name="Unrouted" color="6" fill="1" visible="yes" active="yes"/>
 <layer number="20" name="Dimension" color="15" fill="1" visible="yes" active="yes"/>
-<layer number="21" name="tPlace" color="7" fill="1" visible="no" active="yes"/>
+<layer number="21" name="tPlace" color="7" fill="1" visible="yes" active="yes"/>
 <layer number="22" name="bPlace" color="7" fill="1" visible="yes" active="yes"/>
-<layer number="23" name="tOrigins" color="15" fill="1" visible="no" active="yes"/>
+<layer number="23" name="tOrigins" color="15" fill="1" visible="yes" active="yes"/>
 <layer number="24" name="bOrigins" color="15" fill="1" visible="yes" active="yes"/>
 <layer number="25" name="tNames" color="7" fill="1" visible="no" active="yes"/>
 <layer number="26" name="bNames" color="7" fill="1" visible="no" active="yes"/>
-<layer number="27" name="tValues" color="7" fill="1" visible="no" active="yes"/>
+<layer number="27" name="tValues" color="7" fill="1" visible="yes" active="yes"/>
 <layer number="28" name="bValues" color="7" fill="1" visible="yes" active="yes"/>
 <layer number="29" name="tStop" color="7" fill="3" visible="no" active="yes"/>
@@
 <layer number="31" name="tCream" color="7" fill="4" visible="no" active="yes"/>
 <layer number="32" name="bCream" color="7" fill="5" visible="no" active="yes"/>
-<layer number="33" name="tFinish" color="6" fill="3" visible="no" active="yes"/>
+<layer number="33" name="tFinish" color="6" fill="3" visible="yes" active="yes"/>
 <layer number="34" name="bFinish" color="6" fill="6" visible="yes" active="yes"/>
 <layer number="35" name="tGlue" color="7" fill="4" visible="no" active="yes"/>
@@
 <layer number="49" name="Reference" color="7" fill="1" visible="no" active="yes"/>
 <layer number="50" name="dxf" color="12" fill="1" visible="no" active="no"/>
-<layer number="51" name="tDocu" color="7" fill="1" visible="no" active="yes"/>
+<layer number="51" name="tDocu" color="7" fill="1" visible="yes" active="yes"/>
 <layer number="52" name="bDocu" color="7" fill="1" visible="yes" active="yes"/>
 <layer number="53" name="tGND_GNDA" color="7" fill="1" visible="no" active="no"/>
@@
 <element name="RL1" library="rcl" package="R0805" value="1K" x="12.7" y="24.13" rot="MR180"/>
 <element name="RL7" library="rcl" package="R0805" value="1K" x="12.7" y="29.21" rot="MR180"/>
-<element name="Q1" library="infineon" package="PG-SOT-223" value="BSP613P" x="52.07" y="11.43">
+<element name="Q1" library="infineon" package="PG-SOT-223" value="BSP75" x="52.07" y="11.43">
 <attribute name="OC_NEWARK" value="unknown" x="132.08" y="-50.8" size="1.778" layer="27" display="off"/>
 <attribute name="MPN" value="" x="132.08" y="-50.8" size="1.778" layer="27" display="off"/>
