File: PCB/Linear Sensor/v1.1/linearSensor.sch (EAGLE design)
At the start: 42 parts, among them CON1 SPI, IC1 REG1117, Q1 BSP613P, X3 16MHz, X4 MINI-USB-SCHIELD-32005-201

Commit message: Create new verison
Parts:
- removed USB: BICOLOR-LED, lpatiny:BICOLOR-LED
- added LED1, LED2: GREEN, led:LEDCHIP-LED0805
- D2, D3, D4, D5: value 1N581D1206 -> 1N581
- LED3: device adafruit:LEDCHIP-LED0805 -> led:LEDCHIP-LED0805
- LED4: device lpatiny:LED3MM -> led:LEDCHIP-LED0805
- Q1: value BSP613P -> BSP75
- U$4: value ATMEGA32U4-AU -> 32U4
- X4: value MINI-USB-SCHIELD-32005-201 -> MINI-USB
Connections:
- net D11*: now also U$2.SI2
- net GND: now also LED1.C, LED2.C; no longer USB.C
- net N$14: now also LED1.A; no longer USB.AG
- net N$8: now also LED2.A; no longer USB.AR
Changed lines of the file:
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@@
 <part name="R17" library="rcl" deviceset="R-EU_" device="R0805" value="1k"/>
 <part name="R18" library="rcl" deviceset="R-EU_" device="R1206" value="10k"/>
-<part name="LED3" library="adafruit" deviceset="LED" device="CHIP-LED0805" value="RED"/>
+<part name="LED3" library="led" deviceset="LED" device="CHIP-LED0805" value="RED"/>
 <part name="R27" library="rcl" deviceset="R-EU_" device="R0805" value="1K"/>
 <part name="C5" library="rcl" deviceset="C-EU" device="C1206" value="10uF"/>
@@
 <part name="GND14" library="supply1" deviceset="GND" device=""/>
 <part name="C10" library="rcl" deviceset="C-EU" device="C1206" value="10uF"/>
-<part name="D2" library="lpatiny" deviceset="1N581*" device="D1206" value="1N581D1206"/>
+<part name="D2" library="lpatiny" deviceset="1N581*" device="D1206" value="1N581"/>
 <part name="GND15" library="supply1" deviceset="GND" device=""/>
-<part name="LED4" library="lpatiny" deviceset="LED3MM" device="" value="RED"/>
+<part name="LED4" library="led" deviceset="LED" device="CHIP-LED0805" value="RED"/>
 <part name="RL4" library="resistor" deviceset="R-EU_" device="R0805" value="1K"/>
-<part name="D3" library="lpatiny" deviceset="1N581*" device="D1206" value="1N581D1206"/>
+<part name="D3" library="lpatiny" deviceset="1N581*" device="D1206" value="1N581"/>
 <part name="U$7" library="MyPOW" deviceset="VUSB" device=""/>
 <part name="C12" library="rcl" deviceset="C-EU" device="C1206" value="100nF"/>
-<part name="D4" library="lpatiny" deviceset="1N581*" device="D1206" value="1N581D1206"/>
+<part name="D4" library="lpatiny" deviceset="1N581*" device="D1206" value="1N581"/>
 <part name="GND3" library="supply1" deviceset="GND" device=""/>
-<part name="USB" library="lpatiny" deviceset="BICOLOR-LED" device=""/>
 <part name="RL1" library="rcl" deviceset="R-EU_" device="R0805" value="1K"/>
 <part name="RL7" library="rcl" deviceset="R-EU_" device="R0805" value="1K"/>
 <part name="GND1" library="supply1" deviceset="GND" device=""/>
-<part name="Q1" library="infineon" deviceset="BSP613P" device=""/>
+<part name="Q1" library="infineon" deviceset="BSP613P" device="" value="BSP75"/>
 <part name="GND29" library="supply1" deviceset="GND" device=""/>
 <part name="+5VA2" library="supply1" deviceset="+5V" device=""/>
-<part name="U$4" library="adafruit" deviceset="ATMEGA32U4" device="-AU"/>
+<part name="U$4" library="adafruit" deviceset="ATMEGA32U4" device="-AU" value="32U4"/>
 <part name="GND28" library="supply1" deviceset="GND" device=""/>
 <part name="RESET1" library="lpatiny" deviceset="TAC_SWITCH" device="SMD" value="Reset uC"/>
@@
 <part name="U$8" library="MyPOW" deviceset="VUSB" device=""/>
 <part name="P+4" library="SparkFun" deviceset="3.3V" device=""/>
-<part name="D5" library="lpatiny" deviceset="1N581*" device="D1206" value="1N581D1206"/>
+<part name="D5" library="lpatiny" deviceset="1N581*" device="D1206" value="1N581"/>
 <part name="R3" library="resistor" deviceset="R-EU_" device="M0805" value="10k"/>
 <part name="GND4" library="supply1" deviceset="GND" device=""/>
@@
 <part name="SUPPLY4" library="supply2" deviceset="+5V/1" device=""/>
 <part name="P+11" library="supply1" deviceset="+5V" device=""/>
-<part name="X4" library="con-cypressindustries" deviceset="MINI-USB-SCHIELD-" device="32005-201"/>
+<part name="X4" library="con-cypressindustries" deviceset="MINI-USB-SCHIELD-" device="32005-201" value="MINI-USB"/>
 <part name="R24" library="resistor" deviceset="R-EU_" device="M1206" value="22"/>
 <part name="R31" library="resistor" deviceset="R-EU_" device="M1206" value="22"/>
@@
 <part name="GND5" library="supply1" deviceset="GND" device=""/>
 <part name="C4" library="rcl" deviceset="C-EU" device="C1206" value="100nF"/>
+<part name="LED1" library="led" deviceset="LED" device="CHIP-LED0805" value="GREEN"/>
+<part name="LED2" library="led" deviceset="LED" device="CHIP-LED0805" value="GREEN"/>
 </parts>
 <sheets>
@@
 <instance part="D4" gate="G$1" x="248.92" y="142.24"/>
 <instance part="GND3" gate="1" x="-71.12" y="264.16"/>
-<instance part="USB" gate="G$1" x="-68.58" y="236.22"/>
 <instance part="RL1" gate="G$1" x="-78.74" y="243.84" rot="MR180"/>
 <instance part="RL7" gate="G$1" x="-78.74" y="228.6" rot="MR180"/>
@@
 <instance part="GND5" gate="1" x="193.04" y="238.76"/>
 <instance part="C4" gate="G$1" x="193.04" y="243.84" rot="MR180"/>
+<instance part="LED1" gate="G$1" x="-55.88" y="231.14" rot="R180"/>
+<instance part="LED2" gate="G$1" x="-55.88" y="241.3"/>
 </instances>
 <busses>
@@
 </segment>
 <segment>
-<pinref part="USB" gate="G$1" pin="C"/>
 <wire x1="-71.12" y1="236.22" x2="-76.2" y2="236.22" width="0.1524" layer="91"/>
 <pinref part="GND1" gate="1" pin="GND"/>
+<pinref part="LED1" gate="G$1" pin="C"/>
+<pinref part="LED2" gate="G$1" pin="C"/>
+<wire x1="-55.88" y1="236.22" x2="-71.12" y2="236.22" width="0.1524" layer="91"/>
 </segment>
 <segment>
@@
 <wire x1="213.36" y1="248.92" x2="208.28" y2="248.92" width="0.1524" layer="91"/>
 <label x="205.74" y="248.92" size="1.778" layer="95"/>
+<wire x1="213.36" y1="248.92" x2="226.06" y2="248.92" width="0.1524" layer="91"/>
+<wire x1="226.06" y1="248.92" x2="226.06" y2="241.3" width="0.1524" layer="91"/>
+<pinref part="U$2" gate="G$1" pin="SI2"/>
+<wire x1="226.06" y1="241.3" x2="236.22" y2="241.3" width="0.1524" layer="91"/>
+<junction x="213.36" y="248.92"/>
+<junction x="236.22" y="241.3"/>
 </segment>
 </net>
@@
 <segment>
 <pinref part="RL1" gate="G$1" pin="2"/>
-<pinref part="USB" gate="G$1" pin="AR"/>
 <wire x1="-73.66" y1="243.84" x2="-68.58" y2="243.84" width="0.1524" layer="91"/>
+<pinref part="LED2" gate="G$1" pin="A"/>
+<wire x1="-68.58" y1="243.84" x2="-55.88" y2="243.84" width="0.1524" layer="91"/>
 </segment>
 </net>
 <net name="N$14" class="0">
 <segment>
-<pinref part="USB" gate="G$1" pin="AG"/>
 <pinref part="RL7" gate="G$1" pin="2"/>
 <wire x1="-68.58" y1="228.6" x2="-73.66" y2="228.6" width="0.1524" layer="91"/>
+<pinref part="LED1" gate="G$1" pin="A"/>
+<wire x1="-68.58" y1="228.6" x2="-55.88" y2="228.6" width="0.1524" layer="91"/>
 </segment>
 </net>
@@
 <wire x1="205.74" y1="251.46" x2="193.04" y2="251.46" width="0.1524" layer="91"/>
 <wire x1="193.04" y1="251.46" x2="193.04" y2="248.92" width="0.1524" layer="91"/>
-</segment>
-</net>
+<junction x="205.74" y="251.46"/>
+</segment>
+</net>
