File: PCB/BerthaBluetooth/v1.0b/berthaBluetooth.brd (EAGLE design)
At the start: 111.9 x 84.6 mm, 112 parts, among them CON1 SPI, IC1 REG1117, J1 RJ12, J2 RJ12, J3 RJ12, J4 RJ12, J5 RJ12, J6 RJ12, Q1 BSP75, Q10 BSP75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

Commit message: Update Board
Parts:
- moved D3 43.5 mm to (26.7, 35.6), turned to 180 degrees
- moved D5 22.2 mm to (45.7, 47.0), turned to 90 degrees
- moved R9 7.41 mm to (66.0, 47.0), flipped to the bottom, turned to 0 degrees
- moved R2 4.02 mm to (66.0, 49.5), flipped to the bottom, turned to 0 degrees
- moved C3 2.03 mm to (54.9, 49.5), turned to 180 degrees
- moved U$1 1.27 mm to (55.9, 47.0)
- turned R10 to 180 degrees
- flipped R16 to the top
- flipped R17 to the top
