File: PCB/SolarDecathlon/v1.0/v1.sch (EAGLE design)
At the start: 108 parts, among them CON1 SPI, IC1 REG1117, J1 RJ12, J2 RJ12, J3 RJ12, J4 RJ12, J5 RJ12, J6 RJ12, Q1 BSP75, Q10 BSP75, Q2 BSP75, Q3 BSP75, Q4 BSP75, Q5 BSP75, Q6 BSP75, Q8 BSP75, Q9 BSP75, X3 16MHz, X4 MINI-USB

Commit message: Solar Decathlon v1
Parts:
- removed D5: 1N581D1206, lpatiny:1N581D1206
- removed F1, F2: 0.5A, lpatiny:POLYSWITCHSMD1812
- removed I2C-J1, I2C-J2, I2C-J3, I2C-J4: RJ12STRAIGHT-I2C, lpatiny:RJ12STRAIGHT-I2C
- removed LED10: RED, lpatiny:LED3MM
- removed Q10, Q8, Q9: BSP75, infineon:BSP613P
- removed R1, R16, R18: 10k, rcl:R-EU_R0805
- removed R17: 1k, rcl:R-EU_R0805
- removed R21, R22, R23, R26, R28, R29, R30, R36, R37, R38: 10K, resistor:R-EU_M0805
- removed RGB-J1: RJ12, lpatiny:RJ12STRAIGHT-RGB
- removed RGB_5-6-11: (no value), lpatiny:TOPLED-3
- removed RL1, RL3, RL5, RL6, RL7: 1K, rcl:R-EU_R0805
- removed RL2, RL8, RL9: 1K, resistor:R-EU_M0805
- removed SERIAL: BICOLOR-LED, lpatiny:BICOLOR-LED
- removed U$6: KPJX-4S-S, lpatiny:KPJX-4S-S
- removed USB: BICOLOR-LED COMMON CAT, lpatiny:BICOLOR-LED
- added C4: 100nF, rcl:C-EUC1206
- added C6: 220nF, rcl:C-EUC1206
- added JP1: (no value), SparkFun:M02LOCK_LONGPADS
- added R2, R9: 10k, resistor:R-EU_M1206
- U$1: value SST25VF064C -> M24512; device BertaLib:SST25VF064C -> lpatiny:M24512
- U$2: value PCA9518 -> CHIPCAP; device lpatiny:PCA9518 -> lpatiny:CHIPCAP
Connections:
- net +5V/1 renamed VCC
- removed net FMOSI: D5.A, R1.1, U$1.MOSI
- removed net N$10: R16.1, R17.1, U$1.CS
- removed net N$13: RL5.2, SERIAL.AR
- removed net N$14: RL7.2, USB.AG
- removed net N$15: RL6.2, SERIAL.AG
- removed net N$23: R18.2, U$1.SCK
- removed net N$36: RGB_5-6-11.CRED, RL2.2
- removed net N$37: RGB_5-6-11.CBLUE, RL8.2
- removed net N$38: F2.1, U$6.+5V
- removed net N$39: F1.1, U$6.+12V
- removed net N$40: RGB_5-6-11.CGREEN, RL9.2
- removed net N$50: Q9.D@1, RGB-J1.3, RL8.1
- removed net N$68: Q8.D@1, RGB-J1.2, RL2.1
- removed net N$75: LED10.A, RL3.1
- removed net N$8: RL1.2, USB.AR
- removed net SCL1: I2C-J4.2, R30.2, U$2.SCL1
- removed net SCL2: I2C-J3.2, R37.1, U$2.SCL2
- removed net SCL3: I2C-J2.2, R22.1, U$2.SCL3
- removed net SCL4: I2C-J1.2, R23.1, U$2.SCL4
- removed net SDA1: I2C-J4.3, R36.1, U$2.SDA1
- removed net SDA2: I2C-J3.3, R38.1, U$2.SDA2
- removed net SDA3: I2C-J2.3, R26.1, U$2.SDA3
- removed net SDA4: I2C-J1.3, R21.2, U$2.SDA4
- net +12V: no longer F1.2, I2C-J1.1, I2C-J2.1, I2C-J3.1, I2C-J4.1, RGB-J1.1, RL3.2
- net +5V: now also JP1.1; no longer F2.2, I2C-J1.5, I2C-J2.5, I2C-J3.5, I2C-J4.5, R21.1, R22.2, R23.2, R26.2, R28.1, R29.1, R30.1, R36.2, R37.2, R38.2, RGB-J1.5, RGB_5-6-11.A2
- net 3.3V: now also C6.1, R2.2, R9.1, U$2.VDD; no longer R1.2, R16.2, U$1.HOLD, U$1.WP, U$2.VCC
- net CS: no longer R17.2
- net D12*: no longer Q8.G
- net D13*: no longer Q9.G
- net D7*: no longer Q10.G
- net GND: now also C4.2, C6.2, JP1.2, U$1.-WC, U$1.E0, U$1.E1, U$1.E2, U$1.VSS; no longer I2C-J1.4, I2C-J1.6, I2C-J2.4, I2C-J2.6, I2C-J3.4, I2C-J3.6, I2C-J4.4, I2C-J4.6, LED10.C, Q10.S, Q8.S, Q9.S, RGB-J1.6, SERIAL.C, U$1.GND, U$6.GND1, U$6.GND2, USB.C
- net MISO: no longer U$1.MISO
- net MOSI: no longer D5.C
- net N$6: now also C4.1, U$2.VCORE; no longer Q10.D@1, RGB-J1.4, RL9.1
- net RD+: no longer RL7.1
- net RD-: no longer RL1.1
- net RXLED: no longer RL5.1
- net SCK: no longer R18.1
- net SCL: now also R9.2, U$1.SCL, U$2.SCL; no longer R28.2, U$2.SCL0
- net SDA: now also R2.1, U$1.SDA, U$2.SDA; no longer R29.2, U$2.SDA0
- net TXLED: no longer RL6.1
Other:
- note added: "I2C Memory"
- note added: "ZigBee"
- note removed: "Flash Memory"
- note removed: "RS232 (Bluetooth) & i2c"
- moved on the sheet: U$1

Commit message: Update wiegand
Parts:
- removed J1, J2, J3, J4, J5, J6: RJ12, lpatiny:RJ12STRAIGHT
- removed LED1, LED2, LED5, LED6, LED8: Blue, lpatiny:LED3MM
- removed LED4: RED, lpatiny:LED3MM
- removed LED7: BLue, lpatiny:LED3MM
- removed Q1, Q2, Q4, Q6: BSP75, infineon:BSP613P
- removed R, R19, R20, R25, R32, R33, R34, R35: 1k, rcl:R-EU_R0805
- removed RL4: 1K, resistor:R-EU_R0805
- added C13, C15: 100nF, rcl:C-EUC1206
- added C14: 10uF, rcl:C-EUC1206
- added JP10, JP7, JP8, JP9: (no value), SparkFun:M03LONGPADS
- added JP2, JP3, JP4, JP5, JP6: (no value), SparkFun:M02LOCK_LONGPADS
- added R1: 4.7k, resistor:R-EU_M1206
- added U$5: DS18B20, lpatiny:DS18B20
- added U1: MPL3115A2LGA8, SparkFun-Sensors:MPL3115A2LGA8
- CON1: device lpatiny:TINYISPT -> lpatiny:TINYISPTAG
- R4, R5, R6, R7: value 1k -> 4.7k; device rcl:R-EU_R0805 -> resistor:R-EU_M1206
Connections:
- removed net +12V: J1.1, J2.1, J3.1, J4.1, J5.1, J6.1
- removed net N$1: J3.2, LED6.C, Q4.D@1
- removed net N$12: LED4.A, RL4.2
- removed net N$17: LED2.A, R25.1
- removed net N$18: J1.3, R.2
- removed net N$19: J5.2, LED8.C, Q6.D@1
- removed net N$21: J6.2, LED1.C, Q3.D@1
- removed net N$22: LED6.A, R5.1
- removed net N$28: J2.2, LED5.C, Q2.D@1
- removed net N$29: J4.3, R34.2
- removed net N$3: J6.3, R19.2
- removed net N$30: LED7.A, R6.1
- removed net N$32: J5.3, R35.2
- removed net N$33: LED8.A, R7.1
- removed net N$34: J1.2, LED2.C, Q1.D@1
- removed net N$4: LED5.A, R4.1
- removed net N$5: J4.2, LED7.C, Q5.D@1
- removed net N$7: J3.3, R33.2
- removed net N$9: LED1.A, R20.1
- new net $1: C13.2, C14.2, C15.2, JP3.1, U1.GND
- new net $12: JP2.1, U$1.VSS
- new net $2: C4.2, C6.2, JP4.1, U$2.GND
- new net $3: JP5.1, U$5.GND
- new net GND_CONTROLLED: JP2.2, JP3.2, JP4.2, JP5.2, Q3.D@1, Q5.S
- new net N$13: C15.1, U1.CAP
- new net N$8: JP6.1, U$3.GND
- net +5V: no longer J1.5, J2.5, J3.5, J4.5, J5.5, J6.5, R20.2, R25.2, R4.2, R5.2, R6.2, R7.2
- net 3.3V: now also C13.1, C14.1, JP10.1, JP7.1, JP8.1, JP9.1, R1.1, R4.1, R5.1, R6.1, R7.1, U$5.VDD, U1.VDD, U1.VDDIO
- net A0: now also R4.2, U$5.DQ; no longer R35.1
- net A1: now also JP9.2, R6.2; no longer R33.1
- net A2: now also JP8.2, R5.2; no longer R32.1
- net A3: now also JP7.2, R1.2; no longer R.1
- net A4: now also JP10.2, R7.2; no longer R34.1
- net A5: no longer R19.1
- net D10*: no longer Q3.G
- net D11*: no longer Q6.G
- net D5*: no longer Q5.G
- net D6*: now also Q5.G; no longer Q1.G
- net D8*: now also Q3.G; no longer Q2.G
- net D9*: no longer Q4.G
- net GND: now also JP10.3, JP7.3, JP8.3, JP9.3; no longer C4.2, C6.2, J1.4, J1.6, J2.4, J2.6, J3.4, J3.6, J4.4, J4.6, J5.4, J5.6, J6.4, J6.6, LED4.C, Q1.S, Q2.S, Q4.S, Q5.S, Q6.S, U$1.VSS, U$2.GND, U$3.GND
- net N$2: now also JP6.2, Q5.D@1; no longer J2.3, R32.2
- net SCL: now also U1.SCL
- net SDA: now also U1.SDA
- net VCC: no longer RL4.1
Other:
- note removed: "RJ12"
- moved on the sheet: Q3, Q5, R4, R5, R6, R7
