File: PCB/SolarDecathlon/v1.0/v1.brd (EAGLE design)
At the start: 111.9 x 84.6 mm, 112 parts, among them CON1 SPI, IC1 REG1117, J1 RJ12, J2 RJ12, J3 RJ12, J4 RJ12, J5 RJ12, J6 RJ12, Q1 BSP75, Q10 BSP75, Q2 BSP75, Q3 BSP75, Q4 BSP75, Q5 BSP75, Q6 BSP75, Q8 BSP75, Q9 BSP75, U1 HC_05, X3 16MHz, X4 MINI-USB

Commit message: Solar Decathlon v1
Parts:
- removed D5: 1N581D1206, lpatiny:LED-1206
- removed F1, F2: 0.5A, lpatiny:C1812
- removed I2C-J1, I2C-J2, I2C-J3, I2C-J4: RJ12STRAIGHT-I2C, lpatiny:RJ12-STRAIGHT-I2C
- removed LED10: RED, lpatiny:LED3MM
- removed Q10, Q8, Q9: BSP75, infineon:PG-SOT-223
- removed R1, R16, R18: 10k, rcl:R0805
- removed R10, RL1, RL3, RL5, RL6, RL7: 1K, rcl:R0805
- removed R17: 1k, rcl:R0805
- removed R21, R22, R23, R26, R28, R29, R30, R36, R37, R38: 10K, resistor:M0805
- removed RGB-J1: RJ12, lpatiny:RJ12-STRAIGHT-RGB
- removed RGB_5-6-11: (no value), lpatiny:LED-TRICOLOR-THROUGHHOLE
- removed RL2, RL8, RL9: 1K, resistor:M0805
- removed SERIAL: BICOLOR-LED, lpatiny:BICOLOR-3MM
- removed U$6: KPJX-4S-S, lpatiny:KPJX-4S-S
- removed U1: HC_05, Bluetooth HC-05:BLUETOOTH_SMD
- removed USB: BICOLOR-LED COMMON CAT, lpatiny:BICOLOR-3MM
- added C4: 100nF, rcl:C1206
- added C6: 220nF, rcl:C1206
- added JP1: (no value), SparkFun:1X02_LOCK_LONGPADS
- R2: value 2.2K -> 10k; device rcl:R0805 -> resistor:M1206
- R9: value 1.2K -> 10k; device rcl:R0805 -> resistor:M1206
- U$1: value SST25VF064C -> M24512; device BertaLib:SOIC_8-LEAD -> lpatiny:SO8
- U$2: value PCA9518 -> CHIPCAP; device lpatiny:SO20W -> lpatiny:CHIPCAP
- U$3: value SZ05-ZIGBEE -> SZ05-ZIGBEESMD; device lpatiny:SZ05-ZIGBEE -> lpatiny:SZ05-ZIGBEE3
- moved R9 106.9 mm to (-5.08, -22.9), turned to 0 degrees
- moved R2 100.7 mm to (-5.08, -16.5), turned to 0 degrees
- moved U$1 94.5 mm to (0.00, -30.5), flipped to the top, turned to 0 degrees
- moved U$2 88.1 mm to (-10.2, -30.5), flipped to the top
- moved D3 43.5 mm to (26.7, 35.6), turned to 180 degrees
- moved U$3 5.24 mm to (88.9, 38.1)
- moved C3 2.03 mm to (54.9, 49.5), turned to 180 degrees
Connections:
- net +5V/1 renamed VCC
- removed net D2B5: R2.1, R9.1, U1.2
- removed net FMOSI: D5.A, R1.1, U$1.SI
- removed net N$10: R16.1, R17.1, U$1.CE
- removed net N$13: RL5.2, SERIAL.3
- removed net N$14: RL7.2, USB.1
- removed net N$15: RL6.2, SERIAL.1
- removed net N$23: R18.2, U$1.SCK
- removed net N$36: RGB_5-6-11.RED, RL2.2
- removed net N$37: RGB_5-6-11.BLU, RL8.2
- removed net N$38: F2.1, U$6.+5V
- removed net N$39: F1.1, U$6.+12V
- removed net N$40: RGB_5-6-11.GRN, RL9.2
- removed net N$50: Q9.2, RGB-J1.B, RL8.1
- removed net N$68: Q8.2, RGB-J1.R, RL2.1
- removed net N$70: R10.1, U1.1
- removed net N$75: LED10.A, RL3.1
- removed net N$8: RL1.2, USB.3
- removed net SCL1: I2C-J4.SCL, R30.2, U$2.5
- removed net SCL2: I2C-J3.SCL, R37.1, U$2.8
- removed net SCL3: I2C-J2.SCL, R22.1, U$2.12
- removed net SCL4: I2C-J1.SCL, R23.1, U$2.15
- removed net SDA1: I2C-J4.SDA, R36.1, U$2.6
- removed net SDA2: I2C-J3.SDA, R38.1, U$2.9
- removed net SDA3: I2C-J2.SDA, R26.1, U$2.13
- removed net SDA4: I2C-J1.SDA, R21.2, U$2.16
- net +12V: no longer F1.2, I2C-J1.+12V, I2C-J2.+12V, I2C-J3.+12V, I2C-J4.+12V, RGB-J1.+12V, RL3.2
- net +5V: now also JP1.1; no longer F2.2, I2C-J1.+5V, I2C-J2.+5V, I2C-J3.+5V, I2C-J4.+5V, R21.1, R22.2, R23.2, R26.2, R28.1, R29.1, R30.1, R36.2, R37.2, R38.2, RGB-J1.+5V, RGB_5-6-11.GND
- net 3.3V: now also C6.1, R2.2, R9.1, U$1.8, U$2.3; no longer R1.2, R16.2, U$1.RST/HOLD, U$1.VDD, U$1.WP, U$2.20, U1.12
- net CS: no longer R17.2
- net D12*: no longer Q8.1
- net D13*: no longer Q9.1
- net D7*: no longer Q10.1
- net GND: now also C4.2, C6.2, JP1.2, U$1.1, U$1.2, U$1.3, U$1.4, U$1.7, U$2.2, U$3.SND; no longer I2C-J1.GND1, I2C-J1.GND2, I2C-J2.GND1, I2C-J2.GND2, I2C-J3.GND1, I2C-J3.GND2, I2C-J4.GND1, I2C-J4.GND2, LED10.K, Q10.3, Q8.3, Q9.3, R2.2, RGB-J1.GND1, SERIAL.2, U$1.VSS, U$2.10, U$3.SGND, U$6.GND1, U$6.GND2, U1.13, USB.2
- net GND1: now also U$3.RUN; no longer U$3.RNU
- net MISO: no longer U$1.SO
- net MOSI: no longer D5.C
- net N$6: now also C4.1, U$2.1; no longer Q10.2, RGB-J1.G, RL9.1
- net RD+: no longer RL7.1
- net RD-: no longer RL1.1
- net RX: no longer R10.2
- net RXLED: no longer RL5.1
- net SCK: no longer R18.1
- net SCL: now also R9.2, U$1.6, U$2.8; no longer R28.2, U$2.3
- net SDA: now also R2.1, U$1.5, U$2.7; no longer R29.2, U$2.4
- net TX: no longer R9.2
- net TXLED: no longer RL6.1
Routing:
- net +5V: track 570.8 -> 468.1 mm
- net GND: track 462.8 -> 392.4 mm
- net N$38: track 50.8 -> 0.00 mm, vias 1 -> 0
- net N$39: track 38.8 -> 0.00 mm
- net SDA1: track 29.2 -> 0.00 mm
- net SDA2: track 27.9 -> 0.00 mm
- net SDA3: track 27.9 -> 0.00 mm
- net SDA4: track 27.8 -> 0.00 mm
- net +12V: track 330.8 -> 308.0 mm
- net N$50: track 16.5 -> 0.00 mm
- net N$6: track 15.9 -> 0.00 mm
- net SCL4: track 13.9 -> 0.00 mm
- net SCL2: track 13.9 -> 0.00 mm
- net SCL3: track 13.9 -> 0.00 mm
- net N$68: track 13.4 -> 0.00 mm
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
Commit message: Update wiegand
Parts:
- removed J1, J2, J3, J4, J5, J6: RJ12, lpatiny:RJ12-STRAIGHT
- removed LED1, LED2, LED5, LED6, LED8: Blue, lpatiny:LED3MM
- removed LED4: RED, lpatiny:LED3MM
- removed LED7: BLue, lpatiny:LED3MM
- removed Q1, Q2, Q4, Q6: BSP75, infineon:PG-SOT-223
- removed R, R19, R20, R25, R32, R33, R34, R35: 1k, rcl:R0805
- removed RL4: 1K, resistor:R0805
- added C13, C15: 100nF, rcl:C1206
- added C14: 10uF, rcl:C1206
- added JP10, JP7, JP8, JP9: (no value), SparkFun:1X03_LONGPADS
- added JP2, JP3, JP4, JP5, JP6: (no value), SparkFun:1X02_LOCK_LONGPADS
- added R1: 4.7k, resistor:M1206
- added U$5: DS18B20, lpatiny:SO8
- added U1: MPL3115A2LGA8, SparkFun-Sensors:LGA8
- CON1: device lpatiny:TC2030-MCP-NL -> lpatiny:TC2030-MCP
- R4, R5, R6, R7: value 1k -> 4.7k; device rcl:R0805 -> resistor:M1206
- moved C6 104.2 mm to (62.2, 30.5), flipped to the bottom, turned to 180 degrees
- moved C4 102.4 mm to (62.2, 34.3), flipped to the bottom, turned to 180 degrees
- moved U$1 95.6 mm to (73.7, 30.5), turned to 270 degrees
- moved U$2 95.5 mm to (62.2, 31.8), turned to 270 degrees
- moved R9 77.0 mm to (55.9, 24.1), turned to 90 degrees
- moved R2 76.5 mm to (59.7, 24.1), turned to 270 degrees
- moved Q3 62.1 mm to (66.0, 10.2), turned to 270 degrees
- moved R7 52.0 mm to (38.1, 34.3), flipped to the top, turned to 0 degrees
- moved Q5 49.6 mm to (33.0, 25.4), flipped to the top, turned to 0 degrees
- moved R6 47.4 mm to (26.7, 34.3), flipped to the top, turned to 0 degrees
- moved R5 43.0 mm to (15.2, 34.3), flipped to the top, turned to 0 degrees
- moved D2 41.0 mm to (11.4, 2.54)
- moved C10 38.7 mm to (16.5, 2.54)
- moved C12 38.7 mm to (20.3, 2.54)
- moved D3 38.7 mm to (11.4, 0.00)
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Connections:
- removed net +12V: J1.+12V, J2.+12V, J3.+12V, J4.+12V, J5.+12V, J6.+12V
- removed net N$1: J3.PWM, LED6.K, Q4.2
- removed net N$12: LED4.A, RL4.2
- removed net N$17: LED2.A, R25.1
- removed net N$18: J1.I/O, R.2
- removed net N$19: J5.PWM, LED8.K, Q6.2
- removed net N$21: J6.PWM, LED1.K, Q3.2
- removed net N$22: LED6.A, R5.1
- removed net N$28: J2.PWM, LED5.K, Q2.2
- removed net N$29: J4.I/O, R34.2
- removed net N$3: J6.I/O, R19.2
- removed net N$30: LED7.A, R6.1
- removed net N$32: J5.I/O, R35.2
- removed net N$33: LED8.A, R7.1
- removed net N$34: J1.PWM, LED2.K, Q1.2
- removed net N$4: LED5.A, R4.1
- removed net N$5: J4.PWM, LED7.K, Q5.2
- removed net N$7: J3.I/O, R33.2
- removed net N$9: LED1.A, R20.1
- new net $1: C13.2, C14.2, C15.2, JP3.1, U1.3
- new net $12: JP2.1, U$1.4
- new net $2: C4.2, C6.2, JP4.1, U$2.2
- new net $3: JP5.1, U$5.5
- new net GND_CONTROLLED: JP2.2, JP3.2, JP4.2, JP5.2, Q3.2, Q5.3
- new net N$13: C15.1, U1.2
- new net N$8: JP6.1, U$3.GND
- net +5V: no longer J1.+5V, J2.+5V, J3.+5V, J4.+5V, J5.+5V, J6.+5V, R20.2, R25.2, R4.2, R5.2, R6.2, R7.2
- net 3.3V: now also C13.1, C14.1, JP10.1, JP7.1, JP8.1, JP9.1, R1.1, R4.1, R5.1, R6.1, R7.1, U$5.3, U1.1, U1.4
- net A0: now also R4.2, U$5.4; no longer R35.1
- net A1: now also JP9.2, R6.2; no longer R33.1
- net A2: now also JP8.2, R5.2; no longer R32.1
- net A3: now also JP7.2, R1.2; no longer R.1
- net A4: now also JP10.2, R7.2; no longer R34.1
- net A5: no longer R19.1
- net D10*: no longer Q3.1
- net D11*: no longer Q6.1
- net D5*: no longer Q5.1
- net D6*: now also Q5.1; no longer Q1.1
- net D8*: now also Q3.1; no longer Q2.1
- net D9*: no longer Q4.1
- net GND: now also JP10.3, JP7.3, JP8.3, JP9.3; no longer C4.2, C6.2, J1.GND1, J1.GND2, J2.GND1, J2.GND2, J3.GND1, J3.GND2, J4.GND1, J4.GND2, J5.GND1, J5.GND2, J6.GND1, J6.GND2, LED4.K, Q1.3, Q2.3, Q4.3, Q5.3, Q6.3, U$1.4, U$2.2, U$3.GND
- net N$2: now also JP6.2, Q5.2; no longer J2.I/O, R32.2
- net SCL: now also U1.8
- net SDA: now also U1.7
- net VCC: no longer RL4.1
Routing:
- net +5V: track 468.1 -> 0.00 mm
- net GND: track 392.4 -> 2.43 mm
- net +12V: track 308.0 -> 0.00 mm
- net N$3: track 59.1 -> 0.00 mm
- net N$19: track 26.0 -> 0.00 mm
- net N$34: track 26.0 -> 0.00 mm
- net N$28: track 26.0 -> 0.00 mm
- net N$21: track 26.0 -> 0.00 mm
- net N$1: track 26.0 -> 0.00 mm
- net N$5: track 26.0 -> 0.00 mm
- net D6*: track 24.0 -> 0.00 mm
- net D9*: track 23.7 -> 0.00 mm
- net D5*: track 23.6 -> 0.00 mm
- net D8*: track 23.6 -> 0.00 mm
- net D11*: track 23.5 -> 0.00 mm
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Other:
- board size 111.9 x 84.6 mm -> 91.6 x 46.5 mm
- board text added: "Solar Decathlon v1.0"
- board text removed: "BioReactor"
- board text removed: "Control Board v2"

Commit message: Add routing
Routing:
- net GND: track 2.43 -> 368.3 mm, vias 0 -> 5
- net 3.3V: track 0.00 -> 171.5 mm, vias 0 -> 4
- net VCC: track 0.00 -> 158.4 mm, vias 0 -> 8
- net GND_CONTROLLED: track 0.00 -> 120.3 mm
- net +5V: track 0.00 -> 101.0 mm, vias 0 -> 1
- net SCL: track 0.00 -> 94.2 mm, vias 0 -> 2
- net A3: track 0.00 -> 91.3 mm, vias 0 -> 1
- net SDA: track 0.00 -> 85.1 mm, vias 0 -> 2
- net RESET: track 2.43 -> 76.7 mm, vias 0 -> 2
- net A1: track 0.00 -> 61.0 mm, vias 0 -> 1
- net MISO: track 2.80 -> 61.4 mm, vias 0 -> 3
- net A2: track 0.00 -> 58.6 mm, vias 0 -> 2
- net TX: track 0.00 -> 54.0 mm, vias 0 -> 1
- net VUSB: track 0.00 -> 52.9 mm, vias 0 -> 3
- net SCK: track 3.25 -> 55.2 mm, vias 0 -> 3
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