File: Wiegand/v1.0b/1.0.sch (EAGLE design)
At the start: 64 parts, among them CON1 SPI, IC1 REG1117, Q3 BSP75, Q5 BSP75, U1 MPL3115A2LGA8, X3 16MHz, X4 MINI-USB

Commit message: Update wiegand
Parts:
- removed C1, C14, C5: 10uF, rcl:C-EUC1206
- removed C13, C15, C4: 100nF, rcl:C-EUC1206
- removed C6: 220nF, rcl:C-EUC1206
- removed IC1: REG1117, burr-brown:REG1117
- removed JP1, JP2, JP3, JP4, JP5, JP6: (no value), SparkFun:M02LOCK_LONGPADS
- removed JP10, JP7, JP8, JP9: (no value), SparkFun:M03LONGPADS
- removed LED3: RED, adafruit:LEDCHIP-LED0805
- removed R27: 1K, rcl:R-EU_R0805
- removed R6, R7: 4.7k, resistor:R-EU_M1206
- removed R9: 10k, resistor:R-EU_M1206
- removed U$1: M24512, lpatiny:M24512
- removed U$2: CHIPCAP, lpatiny:CHIPCAP
- removed U$5: DS18B20, lpatiny:DS18B20
- removed U1: MPL3115A2LGA8, SparkFun-Sensors:MPL3115A2LGA8
- added F1, F2: 0.5A, lpatiny:POLYSWITCHSMD1812
- added J1, J2, J3, J4, J5: RJ12, lpatiny:RJ12STR-WIEGAND
- added LED1, LED2, LED5, LED6, LED7: Blue, lpatiny:LED3MM
- added LED10, LED4: RED, lpatiny:LED3MM
- added Q1, Q2, Q4: BSP75, zetex:PNPSOT223
- added R25: 10k, rcl:R-EU_R0805
- added RL3: 1K, rcl:R-EU_R0805
- added RL4: 1K, resistor:R-EU_R0805
- added U$6: KPJX-4S-S, lpatiny:KPJX-4S-S
- Q3, Q5: device infineon:BSP613P -> zetex:PNPSOT223
- R1, R4, R5: value 4.7k -> 10k; device resistor:R-EU_M1206 -> rcl:R-EU_R0805
- R2: device resistor:R-EU_M1206 -> rcl:R-EU_R0805
- U$3: value SZ05-ZIGBEESMD -> SZ05-ZIGBEE; device lpatiny:SZ05-ZIGBEESMD -> lpatiny:SZ05-ZIGBEE
Connections:
- removed net $1: C13.2, C14.2, C15.2, JP3.1, U1.GND
- removed net $12: JP2.1, U$1.VSS
- removed net $2: C4.2, JP4.1, U$2.GND
- removed net $3: JP5.1, U$5.GND
- removed net 3.3V: C1.1, C13.1, C14.1, C6.1, IC1.VOUT, JP10.1, JP7.1, JP8.1, JP9.1, R1.1, R2.2, R27.2, R4.1, R5.1, R6.1, R7.1, R9.1, U$1.VCC, U$2.VDD, U$5.VDD, U1.VDD, U1.VDDIO
- removed net CTRL_GND: C6.2
- removed net GND_CONTROLLED: JP2.2, JP3.2, JP4.2, JP5.2, Q3.D@1, Q5.S
- removed net N$13: C15.1, U1.CAP
- removed net N$2: JP6.2, Q5.D@1
- removed net N$20: LED3.A, R27.1
- removed net N$6: C4.1, U$2.VCORE
- removed net N$8: JP6.1, U$3.GND
- removed net SCL: R9.2, U$1.SCL, U$2.SCL, U$4.PD0(INT0/OC0B/SCL), U1.SCL
- removed net SDA: R2.1, U$1.SDA, U$2.SDA, U$4.PD1(INT1/SDA), U1.SDA
- removed net VCC: C10.1, C12.2, C5.1, D2.C, D3.C, D4.C, IC1.VIN, R15.2, U$4.AVCC, U$4.AVCC1, U$4.UVCC, U$4.VCC, U$4.VCC1
- new net +12V: F1.2, Q1.E, Q2.E, Q3.E, Q4.E, Q5.E, RL3.2
- new net +5V/1: C10.1, C12.2, D2.C, D3.C, D4.C, R15.2, RL4.1, U$4.AVCC, U$4.AVCC1, U$4.UVCC, U$4.VCC, U$4.VCC1
- new net D2*: J1.2, U$4.PD1(INT1/SDA)
- new net D3*: J1.3, U$4.PD0(INT0/OC0B/SCL)
- new net D4*: J2.2
- new net N$1: LED1.A, R1.1
- new net N$12: LED4.A, RL4.2
- new net N$17: LED2.A, R25.1
- new net N$19: LED6.A, R4.1
- new net N$22: J4.1, Q4.C, R4.2
- new net N$23: J1.1, Q1.C, R25.2
- new net N$29: LED7.A, R5.1
- new net N$3: J2.1, Q2.C, R1.2
- new net N$31: J5.1, Q5.C, R5.2
- new net N$38: F2.1, U$6.+5V
- new net N$39: F1.1, U$6.+12V
- new net N$5: LED5.A, R2.1
- new net N$7: J3.1, Q3.C, R2.2
- new net N$75: LED10.A, RL3.1
- net +5V: now also F2.2, J1.5, J2.5, J3.5, J4.5, J5.5; no longer JP1.1
- net A0: now also J5.4; no longer R4.2, U$5.DQ
- net A1: now also J3.4; no longer JP9.2, R6.2
- net A2: now also J2.4; no longer JP8.2, R5.2
- net A3: now also J1.4, J4.4; no longer JP7.2, R1.2
- net A4: no longer JP10.2, R7.2
- net D10*: now also J3.2
- net D11*: now also Q5.B
- net D12*: now also J3.3
- net D13*: now also J4.2
- net D5*: now also Q4.B
- net D6*: now also Q1.B
- net D7*: now also J2.3
- net D8*: now also Q2.B
- net D9*: now also Q3.B; no longer Q3.G, Q5.G
- net GND: now also J1.6, J2.6, J3.6, J4.6, J5.6, LED1.C, LED10.C, LED2.C, LED4.C, LED5.C, LED6.C, LED7.C, U$3.GND, U$6.GND1, U$6.GND2; no longer C1.2, C5.2, IC1.GND, JP1.2, JP10.3, JP7.3, JP8.3, JP9.3, LED3.C, Q3.S, U$1.-WC, U$1.E0, U$1.E1, U$1.E2
- net MISO: now also J4.3
- net MOSI: now also J5.3
- net SCK: now also J5.2
Other:
- note added: "RJ12"
- note added: "RS232 (Bluetooth) & i2c"
- note removed: "I2C Memory"
- note removed: "ZigBee"
- moved on the sheet: R1, R2, R4, R5, U$3
