File: Wiegand/v1.1/1.0.brd (EAGLE design)
At the start: 96.7 x 71.9 mm, 58 parts, among them CON1 SPI, J1 RJ12, J2 RJ12, J3 RJ12, J4 RJ12, J5 RJ12, Q1 BSP75, Q2 BSP75, Q3 BSP75, Q4 BSP75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

Commit message: Update board adding a LED
Parts:
- removed LED7: Blue, lpatiny:LED3MM
- added LED0, LED3: Blue, SparkFun:LED-1206
- added R6: 1K, rcl:R0805
- LED1, LED10, LED2: device lpatiny:LED3MM -> SparkFun:LED-1206
- LED11, LED12, LED9: device adafruit:CHIP-LED0805 -> SparkFun:LED-1206
- LED4: value RED -> Blue; device lpatiny:LED3MM -> SparkFun:LED-1206
- LED5, LED6: value Blue -> RED; device lpatiny:LED3MM -> SparkFun:LED-1206
- Q1, Q2, Q3, Q4, Q5: value BSP75 -> BCP69
- moved LED4 82.1 mm to (88.9, 61.0), turned to 270 degrees
- moved LED6 60.8 mm to (45.7, 6.35), turned to 0 degrees
- moved LED5 56.8 mm to (19.1, 17.8), turned to 180 degrees
- moved LED2 33.0 mm to (55.9, 61.0)
- moved R8 5.24 mm to (74.9, 16.5)
- moved R11 5.24 mm to (77.5, 16.5)
- moved LED12 5.08 mm to (74.9, 27.9), turned to 90 degrees
- moved R39 5.08 mm to (74.9, 22.9)
- moved LED11 5.08 mm to (77.5, 27.9), turned to 90 degrees
- moved LED9 5.08 mm to (80.0, 27.9), turned to 90 degrees
- moved R12 5.08 mm to (80.0, 22.9)
- moved R14 5.08 mm to (77.5, 22.9)
- moved C11 2.54 mm to (54.6, 26.7)
- moved CFG 1.80 mm to (64.8, 22.9)
- moved RL3 1.27 mm to (24.1, 12.7)
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- renumbered J1 to DOOR0, J2 to DOOR1, J3 to DOOR2, J4 to DOOR3, J5 to DOOR4
Connections:
- new net +5V1: R6.2
- new net N$2: LED6.A, R6.1
- net GND: now also LED0.C, LED1.C, LED10.C, LED2.C, LED3.C, LED4.C, LED5.C, LED6.C; no longer LED1.K, LED10.K, LED2.K, LED4.K, LED5.K, LED6.K, LED7.K
- net N$12: now also LED5.A; no longer LED4.A
- net N$17: now also LED0.A; no longer LED2.A
- net N$19: now also LED3.A; no longer LED6.A
- net N$29: now also LED4.A; no longer LED7.A
- net N$5: now also LED2.A; no longer LED5.A
