File: Wiegand/v1.1/1.0.sch (EAGLE design)
At the start: 58 parts, among them CON1 SPI, J1 RJ12, J2 RJ12, J3 RJ12, J4 RJ12, J5 RJ12, Q1 BSP75, Q2 BSP75, Q3 BSP75, Q4 BSP75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

Commit message: Update board adding a LED
Parts:
- removed LED7: Blue, lpatiny:LED3MM
- added LED0, LED3: Blue, SparkFun:LED1206
- added R6: 1K, rcl:R-EU_R0805
- CON1: device lpatiny:TINYISPT -> lpatiny:TINYISPTAG
- LED1, LED10, LED2: device lpatiny:LED3MM -> SparkFun:LED1206
- LED11, LED12, LED9: device adafruit:LEDCHIP-LED0805 -> SparkFun:LED1206
- LED4: value RED -> Blue; device lpatiny:LED3MM -> SparkFun:LED1206
- LED5, LED6: value Blue -> RED; device lpatiny:LED3MM -> SparkFun:LED1206
- Q1, Q2, Q3, Q4, Q5: value BSP75 -> BCP69
- renumbered J1 to DOOR0, J2 to DOOR1, J3 to DOOR2, J4 to DOOR3, J5 to DOOR4
Connections:
- removed net D14*: DOOR3.3, U$4.PB3(PDO/MISO)
- removed net D15*: DOOR4.2, U$4.PB1(SCK)
- removed net D16*: DOOR4.3, U$4.PB2(PDI/MOSI)
- removed net D4*: DOOR1.2
- new net +5V1: R6.2
- new net N$2: LED6.A, R6.1
- net A3: no longer DOOR3.4
- net A4: now also DOOR3.4
- net CS: now also DOOR1.2
- net D11*: no longer Q5.B
- net D12*: now also Q5.B
- net GND: now also LED0.C, LED3.C; no longer LED7.C
- net MISO: now also DOOR3.3, U$4.PB3(PDO/MISO)
- net MOSI: now also DOOR4.3, U$4.PB2(PDI/MOSI)
- net N$12: now also LED5.A; no longer LED4.A
- net N$17: now also LED0.A; no longer LED2.A
- net N$19: now also LED3.A; no longer LED6.A
- net N$29: now also LED4.A; no longer LED7.A
- net N$5: now also LED2.A; no longer LED5.A
- net SCK: now also DOOR4.2, U$4.PB1(SCK)
Other:
- moved on the sheet: LED2, LED4, LED5, LED6
