File: Wiegand/v1.1/wiegand.brd (EAGLE design)
At the start: 96.7 x 71.9 mm, 60 parts, among them CON1 SPI, Q1 BCP69, Q2 BCP69, Q3 BCP69, Q4 BCP69, Q5 BCP69, X3 16MHz, X4 MINI-USB

Commit message: New version based on BSP 75
Parts:
- removed F2: 0.5A, lpatiny:C1812
- removed Q5: BCP69, zetex:SOT223
- added Q7: BSP75, infineon:PG-SOT-223
- Q1, Q2, Q3, Q4: value BCP69 -> BSP75; device zetex:SOT223 -> infineon:PG-SOT-223
- U$4: value ATMEGA32U4-AU -> ATMEGA32U4
- moved Q2 21.6 mm to (53.3, 63.5), flipped to the top, turned to 0 degrees
- moved Q4 21.6 mm to (86.4, 63.5), flipped to the top, turned to 0 degrees
- moved Q1 21.6 mm to (36.8, 63.5), flipped to the top, turned to 0 degrees
- moved Q3 21.6 mm to (69.8, 63.5), flipped to the top, turned to 0 degrees
- moved LED2 8.89 mm to (47.0, 61.0), turned to 180 degrees
- moved LED3 8.89 mm to (63.5, 61.0), turned to 180 degrees
- moved LED4 8.89 mm to (80.0, 61.0), turned to 180 degrees
- moved LED0 8.89 mm to (14.0, 61.0), turned to 180 degrees
- moved LED1 8.89 mm to (30.5, 61.0), turned to 180 degrees
- moved R2 6.84 mm to (47.0, 64.8), flipped to the top
- moved R25 6.84 mm to (14.0, 64.8), flipped to the top
- moved R1 6.84 mm to (30.5, 64.8), flipped to the top
- moved R4 6.84 mm to (63.5, 64.8), flipped to the top
- moved R5 6.84 mm to (80.0, 64.5), flipped to the top
Connections:
- removed net N$17: LED0.A, R25.1
- removed net N$19: LED3.A, R4.1
- removed net N$29: LED4.A, R5.1
- removed net N$38: F2.1, U$6.+5V
- new net N$6: LED2.C, R2.1
- new net N$8: LED3.C, R4.1
- new net N$9: LED4.C, R5.1
- net +12V: now also DOOR0.+12V, DOOR1.+12V, DOOR2.+12V, DOOR3.+12V, DOOR4.+12V, LED0.A, LED1.A, LED2.A, LED3.A, LED4.A; no longer Q1.3, Q2.3, Q3.3, Q4.3, Q5.3
- net +5V: now also U$6.+5V; no longer DOOR0.+5V, DOOR1.+5V, DOOR2.+5V, DOOR3.+5V, DOOR4.+5V, F2.2
- net D11*: now also Q4.1
- net D12*: no longer Q5.1
- net D5*: now also Q3.1; no longer Q4.1
- net D6*: now also Q7.1; no longer Q1.1
- net D8*: now also Q1.1; no longer Q2.1
- net D9*: now also Q2.1; no longer Q3.1
- net GND: now also Q1.3, Q2.3, Q3.3, Q4.3, Q7.3; no longer LED0.C, LED1.C, LED2.C, LED3.C, LED4.C
- net N$1: now also LED0.C, R25.1; no longer LED1.A, R1.1
- net N$22: now also DOOR3.PWM, Q3.2; no longer DOOR3.+12V, Q4.2, Q4.4
- net N$23: now also DOOR0.PWM, Q7.2; no longer DOOR0.+12V, Q1.2, Q1.4
- net N$3: now also DOOR1.PWM, Q1.2; no longer DOOR1.+12V, Q2.2, Q2.4
- net N$31: now also DOOR4.PWM, Q4.2; no longer DOOR4.+12V, Q5.2, Q5.4
- net N$5: now also LED1.C, R1.1; no longer LED2.A, R2.1
- net N$7: now also DOOR2.PWM, Q2.2; no longer DOOR2.+12V, Q3.2, Q3.4
Routing:
- net GND: track 232.5 -> 554.1 mm, vias 0 -> 9
- net MOSI: track 3.57 -> 123.6 mm, vias 0 -> 3
- net +12V: track 239.5 -> 356.4 mm, vias 0 -> 1
- net D12*: track 0.00 -> 114.1 mm, vias 0 -> 2
- net MISO: track 2.80 -> 112.3 mm, vias 0 -> 4
- net D9*: track 0.00 -> 109.0 mm, vias 0 -> 4
- net SCK: track 3.57 -> 107.7 mm, vias 0 -> 6
- net D8*: track 0.94 -> 91.7 mm, vias 0 -> 4
- net RESET: track 2.43 -> 82.0 mm, vias 0 -> 6
- net A0: track 0.00 -> 79.0 mm, vias 0 -> 1
- net D11*: track 0.00 -> 76.5 mm, vias 0 -> 2
- net +5V: track 168.9 -> 93.3 mm
- net A4: track 0.00 -> 74.3 mm, vias 0 -> 3
- net +5V/1: track 0.00 -> 73.6 mm, vias 0 -> 4
- net D6*: track 0.00 -> 71.4 mm, vias 0 -> 4
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Other:
- board text added: "Wiegand v1.1"
