File: PCB/IntegratedBertha/v1.0/berthaBluetooth.sch (EAGLE design)
At the start: 55 parts, among them CON1 SPI, Q1 BSP75, Q2 BSP75, Q4 BSP75, Q7 BSP75, X3 16MHz, X4 MINI-USB

Commit message: Add relay card and integrated bioreactor
Parts:
- removed DOOR0, DOOR1, DOOR2, DOOR4: RJ12, lpatiny:RJ12STR-WIEGAND
- removed F1: 0.5A, lpatiny:POLYSWITCHSMD1812
- removed LED0: Blue, SparkFun:LED1206
- added C1, C5: 10uF, rcl:C-EUC1206
- added C4: 100nF, rcl:C-EUC1206
- added C6: 330nF, rcl:C-EUC1206
- added D5: 1N581D1206, lpatiny:1N581D1206
- added I2C-J4: RJ12STRAIGHT-I2C, lpatiny:RJ12STRAIGHT-I2C
- added IC1: REG1117, burr-brown:REG1117
- added IC2: AD8223, analog-devices:AD620R
- added J1, J2, J3, J4, J5: RJ12, lpatiny:RJ12STRAIGHT
- added J7: 22--02, lpatiny:22--02
- added LED13, LED3: RED, adafruit:LEDCHIPLED_1206
- added LED14: GREEN, adafruit:LEDCHIPLED_1206
- added LED7: BLue, adafruit:LEDCHIPLED_1206
- added LED8: Blue, adafruit:LEDCHIPLED_1206
- added Q5, Q6: BSP75, infineon:BSP613P
- added R, R17, R32, R33, R34, R35, R4, R7: 1k, rcl:R-EU_R0805
- added R10, R21: 4.7k, resistor:R-EU_R1206
- added R16, R18: 10k, rcl:R-EU_R0805
- added R27, RL1, RL2, RL5, RL6, RL7, RL8: 1K, rcl:R-EU_R0805
- added R28, R29: 10K, resistor:R-EU_M0805
- added R9: 100, resistor:R-EU_R1206
- added U$1: SST25VF064C, BertaLib:SST25VF064C
- added X1: 22-23-20415.08S, lpatiny:22-23-20415.08S
- added X2, X5: 22-23-20315.08S, lpatiny:22-23-20315.08S
- CON1: device lpatiny:TINYISPTAG -> lpatiny:TINYISPT
- LED1: value Blue -> GREEN; device SparkFun:LED1206 -> adafruit:LEDCHIPLED_1206
- LED10, LED11, LED12, LED2, LED9: device SparkFun:LED1206 -> adafruit:LEDCHIPLED_1206
- LED4: value Blue -> RED; device SparkFun:LED1206 -> adafruit:LEDCHIPLED_1206
- LED5, LED6: value RED -> Blue; device SparkFun:LED1206 -> adafruit:LEDCHIPLED_1206
- Q7: value BSP75 -> IRF3704S; device infineon:BSP613P -> transistor-power:IRF3704S
- R2: value 10k -> 300; device rcl:R-EU_R0805 -> resistor:R-EU_R1206
- R25, R5: value 10k -> 1k
- R6: value 1K -> 1k
- U$4: value ATMEGA32U4 -> ATMEGA32U4-AU
Connections:
- removed net +5V1: R6.2
- removed net D2*: DOOR0.2, U$4.PD1(INT1/SDA)
- removed net D3*: DOOR0.3, U$4.PD0(INT0/OC0B/SCL)
- removed net N$31: DOOR4.5, Q4.D@1, R5.2
- removed net N$39: F1.1, U$6.+12V
- new net 3.3V: C1.1, IC1.VOUT, R1.2, R16.2, R27.2, U$1.HOLD, U$1.VCC, U$1.WP
- new net DIFF+: IC2.+, X1-3.S
- new net DIFF-: IC2.-, X1-2.S
- new net FMOSI: D5.A, R1.1, U$1.MOSI
- new net N$10: R16.1, R17.1, U$1.CS
- new net N$13: IC2.RG@1, R2.2
- new net N$14: LED14.A, RL7.2
- new net N$15: IC2.RG@2, R2.1
- new net N$17: LED2.A, R25.1
- new net N$18: J1.3, R.2
- new net N$19: J5.2, LED8.C, Q6.D@1
- new net N$20: LED3.A, R27.1
- new net N$21: R10.2, RL6.2, X2-2.S
- new net N$22: LED6.A, R5.1
- new net N$28: J2.2, LED5.C, Q2.D@1
- new net N$29: J4.3, R34.2
- new net N$30: LED7.A, R6.1
- new net N$32: J5.3, R35.2
- new net N$33: LED8.A, R7.1
- new net N$34: J1.2, LED2.C, Q1.D@1
- new net N$36: J7-2.S, Q7.D
- new net N$4: LED5.A, R4.1
- new net N$40: IC2.OUT, R9.1
- new net N$8: LED13.A, RL1.2
- new net SCL: I2C-J4.2, R28.2, U$4.PD0(INT0/OC0B/SCL)
- new net SDA: I2C-J4.3, R29.2, U$4.PD1(INT1/SDA)
- net +12V: now also I2C-J4.1, J1.1, J2.1, J3.1, J4.1, J5.1, J7-1.S, U$6.+12V; no longer DOOR0.1, DOOR1.1, DOOR2.1, DOOR4.1, F1.2, LED0.A, LED1.A, LED2.A, LED4.A
- net +5V: now also C4.1, I2C-J4.5, IC2.+V, J1.5, J2.5, J3.5, J4.5, J5.5, R10.1, R21.1, R25.2, R28.1, R29.1, R4.2, R5.2, R6.2, R7.2, X1-1.S, X2-1.S, X5-1.S
- net +5V/1: now also C5.1, IC1.VIN
- net A0: now also R35.1; no longer DOOR4.4
- net A1: now also R33.1; no longer DOOR2.4
- net A2: now also R32.1; no longer DOOR1.4
- net A3: now also R.1; no longer DOOR0.4
- net A4: now also R34.1
- net A5: now also RL8.1
- net CS: now also R17.2
- net D10*: now also RL6.1; no longer DOOR2.2
- net D11*: now also Q6.G; no longer DOOR2.3
- net D12*: now also C6.1, R9.2; no longer Q4.G
- net D13*: now also RL5.1; no longer Q2.G
- net D5*: now also Q5.G; no longer Q1.G
- net D6*: now also Q1.G; no longer Q7.G
- net D7*: now also RL2.1
- net D8*: now also Q2.G; no longer DOOR1.2
- net D9*: now also Q4.G; no longer DOOR1.3
- net GND: now also C1.2, C4.2, C5.2, C6.2, I2C-J4.4, I2C-J4.6, IC1.GND, IC2.-V, IC2.REF, J1.4, J1.6, J2.4, J2.6, J3.4, J3.6, J4.4, J4.6, J5.4, J5.6, LED1.C, LED13.C, LED14.C, LED3.C, LED4.C, Q5.S, Q6.S, U$1.GND, X1-4.S, X2-3.S, X5-3.S; no longer DOOR0.6, DOOR1.6, DOOR2.6, DOOR4.6, LED5.C, LED6.C
- net MISO: now also U$1.MISO; no longer DOOR4.3
- net MOSI: now also D5.C
- net N$1: now also J3.2, LED6.C, Q4.D@1; no longer LED0.C, R25.1
- net N$12: now also LED4.A; no longer LED5.A
- net N$2: now also J2.3, R32.2; no longer LED6.A, R6.1
- net N$23: now also R18.2, U$1.SCK; no longer DOOR0.5, Q7.D@1, R25.2
- net N$3: now also LED1.A, RL5.2; no longer DOOR1.5, Q1.D@1, R1.2
- net N$5: now also J4.2, LED7.C, Q5.D@1; no longer LED1.C, R1.1
- net N$6: now also Q7.G, RL2.2; no longer LED2.C, R2.1
- net N$7: now also J3.3, R33.2; no longer DOOR2.5, Q2.D@1, R2.2
- net N$9: now also R21.2, RL8.2, X5-2.S; no longer LED4.C, R5.1
- net RD+: now also RL7.1
- net RD-: now also RL1.1
- net SCK: now also R18.1; no longer DOOR4.2
Other:
- note added: "Flash Memory"
- note added: "One wire"
- note added: "PID"
- note added: "Weight"
- moved on the sheet: LED1, LED2, LED4, LED5, LED6, Q1, Q2, Q4, R1, R2, R25, R5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
