File: PCB/IntegratedBertha/v1.0/integratedBertha.sch (EAGLE design)
At the start: 97 parts, among them CON1 SPI, IC1 REG1117, IC2 AD8223, J1 RJ12, J2 RJ12, J3 RJ12, J4 RJ12, J5 RJ12, J6 RJ12, J7 22--02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

Commit message: Update integrated
Parts:
- removed J6: RJ12, lpatiny:RJ12STRAIGHT
- removed Q3: BSP75, infineon:BSP613P
- removed R19, R20: 1k, rcl:R-EU_R0805
- added RL5, RL6, RL8: 1K, rcl:R-EU_R0805
- LED1: value Blue -> GREEN
Connections:
- removed net N$31: RL2.1
- removed net N$37: R10.1, X2-1.S
- removed net N$38: IC2.-, X1-1.S
- removed net N$39: IC2.+, X1-2.S
- removed net N$41: R21.1, X5-1.S
- removed net SIGN: C6.1, R9.2
- new net DIFF+: IC2.+, X1-3.S
- new net DIFF-: IC2.-, X1-2.S
- net +12V: no longer J6.1
- net +5V: now also R10.1, R21.1, X1-1.S, X2-1.S, X5-1.S; no longer J6.5, R10.2, R20.2, R21.2, X1-4.S, X2-2.S, X5-2.S
- net A5: now also RL8.1; no longer R19.1
- net D10*: now also RL6.1; no longer Q3.G
- net D12*: now also C6.1, R9.2
- net D13*: now also RL5.1
- net D7*: now also RL2.1
- net GND: now also LED1.C, X1-4.S; no longer J6.4, J6.6, Q3.S, X1-3.S
- net N$21: now also R10.2, RL6.2, X2-2.S; no longer J6.2, LED1.C, Q3.D@1
- net N$3: now also LED1.A, RL5.2; no longer J6.3, R19.2
- net N$9: now also R21.2, RL8.2, X5-2.S; no longer LED1.A, R20.1
Other:
- note added: "One wire"
- note added: "PID"
- note added: "Weight"
- note removed: "analog ????????????"
- moved on the sheet: LED1, R10, R21
