File: PCB/TestZigbeeBlueTooth/v1.0b/berthaBluetooth.sch (EAGLE design)
At the start: 55 parts, among them CON1 SPI, Q1 BSP75, Q2 BSP75, Q4 BSP75, Q7 BSP75, X3 16MHz, X4 MINI-USB

Commit message: Add relay card and integrated bioreactor
Parts:
- removed DOOR0, DOOR1, DOOR2, DOOR4: RJ12, lpatiny:RJ12STR-WIEGAND
- removed LED0: Blue, SparkFun:LED1206
- removed Q7: BSP75, infineon:BSP613P
- removed R2: 10k, rcl:R-EU_R0805
- added C1, C5: 10uF, rcl:C-EUC1206
- added D5: 1N581D1206, lpatiny:1N581D1206
- added F2: 0.5A, lpatiny:POLYSWITCHSMD1812
- added I2C-J1, I2C-J2, I2C-J3, I2C-J4: RJ12STRAIGHT-I2C, lpatiny:RJ12STRAIGHT-I2C
- added IC1: REG1117, burr-brown:REG1117
- added J1, J2, J3, J4, J5, J6: RJ12, lpatiny:RJ12STRAIGHT
- added LED3: RED, adafruit:LEDCHIP-LED0805
- added LED7: BLue, lpatiny:LED3MM
- added LED8: Blue, lpatiny:LED3MM
- added Q10, Q3, Q5, Q6, Q8, Q9: BSP75, infineon:BSP613P
- added R, R17, R19, R20, R32, R33, R34, R35, R4, R7: 1k, rcl:R-EU_R0805
- added R16, R18: 10k, rcl:R-EU_R0805
- added R21, R22, R23, R26, R28, R29, R30, R36, R37, R38: 10K, resistor:R-EU_M0805
- added R27, RL1, RL5, RL6, RL7: 1K, rcl:R-EU_R0805
- added RGB-J1: RJ12, lpatiny:RJ12STRAIGHT-RGB
- added RGB_5-6-11: (no value), lpatiny:TOPLED-3
- added RL2, RL8, RL9: 1K, resistor:R-EU_M0805
- added SERIAL: BICOLOR-LED, lpatiny:BICOLOR-LED
- added U$1: SST25VF064C, BertaLib:SST25VF064C
- added U$2: PCA9518, lpatiny:PCA9518
- added USB: BICOLOR-LED COMMON CAT, lpatiny:BICOLOR-LED
- CON1: device lpatiny:TINYISPTAG -> lpatiny:TINYISPT
- LED1, LED10, LED2: device SparkFun:LED1206 -> lpatiny:LED3MM
- LED11, LED12, LED9: device SparkFun:LED1206 -> adafruit:LEDCHIP-LED0805
- LED4: value Blue -> RED; device SparkFun:LED1206 -> lpatiny:LED3MM
- LED5, LED6: value RED -> Blue; device SparkFun:LED1206 -> lpatiny:LED3MM
- R25, R5: value 10k -> 1k
- R6: value 1K -> 1k
- U$3: value SZ05-ZIGBEE -> SZ05-ZIGBEESMD; device lpatiny:SZ05-ZIGBEE -> lpatiny:SZ05-ZIGBEESMD
- U$4: value ATMEGA32U4 -> ATMEGA32U4-AU
Connections:
- removed net +5V1: R6.2
- removed net D2*: DOOR0.2, U$4.PD1(INT1/SDA)
- removed net D3*: DOOR0.3, U$4.PD0(INT0/OC0B/SCL)
- removed net N$31: DOOR4.5, Q4.D@1, R5.2
- new net 3.3V: C1.1, IC1.VOUT, R1.2, R16.2, R27.2, U$1.HOLD, U$1.VCC, U$1.WP, U$2.VCC
- new net FMOSI: D5.A, R1.1, U$1.MOSI
- new net N$10: R16.1, R17.1, U$1.CS
- new net N$13: RL5.2, SERIAL.AR
- new net N$14: RL7.2, USB.AG
- new net N$15: RL6.2, SERIAL.AG
- new net N$17: LED2.A, R25.1
- new net N$18: J1.3, R.2
- new net N$19: J5.2, LED8.C, Q6.D@1
- new net N$20: LED3.A, R27.1
- new net N$21: J6.2, LED1.C, Q3.D@1
- new net N$22: LED6.A, R5.1
- new net N$28: J2.2, LED5.C, Q2.D@1
- new net N$29: J4.3, R34.2
- new net N$30: LED7.A, R6.1
- new net N$32: J5.3, R35.2
- new net N$33: LED8.A, R7.1
- new net N$34: J1.2, LED2.C, Q1.D@1
- new net N$36: RGB_5-6-11.CRED, RL2.2
- new net N$37: RGB_5-6-11.CBLUE, RL8.2
- new net N$38: F2.1, U$6.+5V
- new net N$4: LED5.A, R4.1
- new net N$40: RGB_5-6-11.CGREEN, RL9.2
- new net N$50: Q9.D@1, RGB-J1.3, RL8.1
- new net N$68: Q8.D@1, RGB-J1.2, RL2.1
- new net N$8: RL1.2, USB.AR
- new net SCL: R28.2, U$2.SCL0, U$4.PD0(INT0/OC0B/SCL)
- new net SCL1: I2C-J4.2, R30.2, U$2.SCL1
- new net SCL2: I2C-J3.2, R37.1, U$2.SCL2
- new net SCL3: I2C-J2.2, R22.1, U$2.SCL3
- new net SCL4: I2C-J1.2, R23.1, U$2.SCL4
- new net SDA: R29.2, U$2.SDA0, U$4.PD1(INT1/SDA)
- new net SDA1: I2C-J4.3, R36.1, U$2.SDA1
- new net SDA2: I2C-J3.3, R38.1, U$2.SDA2
- new net SDA3: I2C-J2.3, R26.1, U$2.SDA3
- new net SDA4: I2C-J1.3, R21.2, U$2.SDA4
- net +12V: now also I2C-J1.1, I2C-J2.1, I2C-J3.1, I2C-J4.1, J1.1, J2.1, J3.1, J4.1, J5.1, J6.1, RGB-J1.1; no longer DOOR0.1, DOOR1.1, DOOR2.1, DOOR4.1, LED0.A, LED1.A, LED2.A, LED4.A
- net +5V: now also F2.2, I2C-J1.5, I2C-J2.5, I2C-J3.5, I2C-J4.5, J1.5, J2.5, J3.5, J4.5, J5.5, J6.5, R20.2, R21.1, R22.2, R23.2, R25.2, R26.2, R28.1, R29.1, R30.1, R36.2, R37.2, R38.2, R4.2, R5.2, R6.2, R7.2, RGB-J1.5, RGB_5-6-11.A2; no longer U$6.+5V
- net +5V/1: now also C5.1, IC1.VIN
- net A0: now also R35.1; no longer DOOR4.4
- net A1: now also R33.1; no longer DOOR2.4
- net A2: now also R32.1; no longer DOOR1.4
- net A3: now also R.1; no longer DOOR0.4
- net A4: now also R34.1
- net A5: now also R19.1
- net CS: now also R17.2
- net D10*: now also Q3.G; no longer DOOR2.2
- net D11*: now also Q6.G; no longer DOOR2.3
- net D12*: now also Q8.G; no longer Q4.G
- net D13*: now also Q9.G; no longer Q2.G
- net D5*: now also Q5.G; no longer Q1.G
- net D6*: now also Q1.G; no longer Q7.G
- net D7*: now also Q10.G
- net D8*: now also Q2.G; no longer DOOR1.2
- net D9*: now also Q4.G; no longer DOOR1.3
- net GND: now also C1.2, C5.2, I2C-J1.4, I2C-J1.6, I2C-J2.4, I2C-J2.6, I2C-J3.4, I2C-J3.6, I2C-J4.4, I2C-J4.6, IC1.GND, J1.4, J1.6, J2.4, J2.6, J3.4, J3.6, J4.4, J4.6, J5.4, J5.6, J6.4, J6.6, LED3.C, LED4.C, Q10.S, Q3.S, Q5.S, Q6.S, Q8.S, Q9.S, RGB-J1.6, SERIAL.C, U$1.GND, U$2.GND, USB.C; no longer DOOR0.6, DOOR1.6, DOOR2.6, DOOR4.6, LED5.C, LED6.C, Q7.S
- net MISO: now also U$1.MISO; no longer DOOR4.3
- net MOSI: now also D5.C
- net N$1: now also J3.2, LED6.C, Q4.D@1; no longer LED0.C, R25.1
- net N$12: now also LED4.A; no longer LED5.A
- net N$2: now also J2.3, R32.2; no longer LED6.A, R6.1
- net N$23: now also R18.2, U$1.SCK; no longer DOOR0.5, Q7.D@1, R25.2
- net N$3: now also J6.3, R19.2; no longer DOOR1.5, Q1.D@1, R1.2
- net N$5: now also J4.2, LED7.C, Q5.D@1; no longer LED1.C, R1.1
- net N$6: now also Q10.D@1, RGB-J1.4, RL9.1; no longer LED2.C, R2.1
- net N$7: now also J3.3, R33.2; no longer DOOR2.5, Q2.D@1, R2.2
- net N$9: now also LED1.A, R20.1; no longer LED4.C, R5.1
- net RD+: now also RL7.1
- net RD-: now also RL1.1
- net RXLED: now also RL5.1
- net SCK: now also R18.1; no longer DOOR4.2
- net TXLED: now also RL6.1
Other:
- note added: "Flash Memory"
- moved on the sheet: LED1, LED2, LED4, LED5, LED6, Q1, Q2, Q4, R1, R25, R5, R6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
