File: Wiegand/v2.0/wiegand.brd (EAGLE design)
At the start: 96.7 x 71.9 mm, 55 parts, among them CON1 SPI, Q1 BSP75, Q2 BSP75, Q4 BSP75, Q7 BSP75, X3 16MHz, X4 MINI-USB

Commit message: Add relay card and integrated bioreactor
Parts:
- removed DOOR0, DOOR1, DOOR2, DOOR4: RJ12, lpatiny:RJ12-STRAIGHT-WIEGAND
- removed LED1, LED2, LED4: Blue, SparkFun:LED-1206
- removed Q1, Q2, Q4: BSP75, infineon:PG-SOT-223
- removed R5: 10k, rcl:R0805
- added X1: 22-23-2071, con-molex:22-23-2071
- added X2, X5: 22-23-2021, con-molex:22-23-2021
- R2: value 10k -> 1k
- moved R2 103.9 mm to (-5.08, -16.5)
- moved R1 89.1 mm to (-5.08, -10.2)
- moved Q7 22.2 mm to (24.1, 43.2)
- moved LED0 22.2 mm to (17.8, 40.6)
- moved R25 22.2 mm to (17.8, 44.5)
Connections:
- removed net N$31: DOOR4.PWM, Q4.2, R5.2
- removed net N$7: DOOR2.PWM, Q2.2, R2.2
- removed net N$9: LED4.C, R5.1
- new net N$4: X1.7
- net +12V: now also X2.2; no longer DOOR0.+12V, DOOR1.+12V, DOOR2.+12V, DOOR4.+12V, LED1.A, LED2.A, LED4.A
- net +5V: now also R1.1
- net A0: no longer DOOR4.I/O
- net A1: no longer DOOR2.I/O
- net A2: now also X5.2; no longer DOOR1.I/O
- net A3: now also R2.1; no longer DOOR0.I/O
- net D10*: no longer DOOR2.DAT0
- net D11*: no longer DOOR2.DAT1
- net D12*: no longer Q4.1
- net D13*: no longer Q2.1
- net D2*: no longer DOOR0.DAT0
- net D3*: no longer DOOR0.DAT1
- net D5*: no longer Q1.1
- net D8*: no longer DOOR1.DAT0
- net D9*: no longer DOOR1.DAT1
- net GND: no longer DOOR0.GND, DOOR1.GND, DOOR2.GND, DOOR4.GND, Q1.3, Q2.3, Q4.3
- net MISO: no longer DOOR4.DAT1
- net N$23: now also X2.1; no longer DOOR0.PWM
- net N$3: now also X1.5; no longer DOOR1.PWM, Q1.2, R1.2
- net N$5: now also R1.2, X5.1; no longer LED1.C, R1.1
- net N$6: now also R2.2, X1.4; no longer LED2.C, R2.1
- net SCK: no longer DOOR4.DAT0
Routing:
- net +12V: track 302.5 -> 128.5 mm
- net GND: track 269.0 -> 144.6 mm
- net N$7: track 14.9 -> 0.00 mm
- net N$3: track 14.9 -> 0.00 mm
- net N$31: track 14.6 -> 0.00 mm
- net N$23: track 14.9 -> 9.77 mm
- net N$6: track 4.36 -> 0.00 mm
- net N$5: track 4.36 -> 0.00 mm
- net N$9: track 4.04 -> 0.00 mm
