File: PCB/IntegratedBertha/v1.0b/integratedBertha.brd (EAGLE design)
At the start: 111.9 x 84.6 mm, 96 parts, among them CON1 SPI, IC1 REG1117, IC2 AD8223, J1 RJ12, J2 RJ12, J3 RJ12, J4 RJ12, J5 RJ12, J7 22--02, Q1 BSP75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

Commit message: Update integrated
Parts:
- moved R12 1.27 mm to (95.2, 36.8)
- moved R14 1.27 mm to (92.7, 36.8)
- moved R39 1.27 mm to (90.2, 36.8)
- moved R11 1.27 mm to (92.7, 31.8)
- moved R8 1.27 mm to (90.2, 31.8)
Connections:
- net +5V: now also X1.1
- net GND: now also X1.4; no longer X1.1
Other:
- board size 111.9 x 84.6 mm -> 108.1 x 84.6 mm
- board text added: "+"
- board text added: "-"
- board text removed: "XX"

Commit message: Upate anemometer
Parts:
- moved C3 2.62 mm to (52.4, 48.9)
Routing:
- net RD-: track 0.00 -> 30.1 mm
- net RD+: track 0.00 -> 30.0 mm
- net D+USB: track 0.00 -> 26.1 mm
- net D-USB: track 0.00 -> 25.9 mm
- net N$16: track 0.00 -> 7.56 mm
- net GND: track 404.4 -> 409.8 mm
Changed lines of the file:
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@@
 <layer number="24" name="bOrigins" color="15" fill="1" visible="yes" active="yes"/>
 <layer number="25" name="tNames" color="7" fill="1" visible="yes" active="yes"/>
-<layer number="26" name="bNames" color="7" fill="1" visible="no" active="yes"/>
+<layer number="26" name="bNames" color="7" fill="1" visible="yes" active="yes"/>
 <layer number="27" name="tValues" color="7" fill="1" visible="yes" active="yes"/>
-<layer number="28" name="bValues" color="7" fill="1" visible="yes" active="yes"/>
+<layer number="28" name="bValues" color="7" fill="1" visible="no" active="yes"/>
 <layer number="29" name="tStop" color="7" fill="3" visible="no" active="yes"/>
 <layer number="30" name="bStop" color="7" fill="6" visible="no" active="yes"/>
 <layer number="31" name="tCream" color="7" fill="4" visible="no" active="yes"/>
 <layer number="32" name="bCream" color="7" fill="5" visible="no" active="yes"/>
-<layer number="33" name="tFinish" color="6" fill="3" visible="yes" active="yes"/>
-<layer number="34" name="bFinish" color="6" fill="6" visible="yes" active="yes"/>
+<layer number="33" name="tFinish" color="6" fill="3" visible="no" active="yes"/>
+<layer number="34" name="bFinish" color="6" fill="6" visible="no" active="yes"/>
 <layer number="35" name="tGlue" color="7" fill="4" visible="no" active="yes"/>
 <layer number="36" name="bGlue" color="7" fill="5" visible="no" active="yes"/>
@@
 <layer number="39" name="tKeepout" color="4" fill="11" visible="no" active="yes"/>
 <layer number="40" name="bKeepout" color="1" fill="11" visible="no" active="yes"/>
-<layer number="41" name="tRestrict" color="4" fill="10" visible="yes" active="yes"/>
-<layer number="42" name="bRestrict" color="1" fill="10" visible="yes" active="yes"/>
-<layer number="43" name="vRestrict" color="2" fill="10" visible="yes" active="yes"/>
+<layer number="41" name="tRestrict" color="4" fill="10" visible="no" active="yes"/>
+<layer number="42" name="bRestrict" color="1" fill="10" visible="no" active="yes"/>
+<layer number="43" name="vRestrict" color="2" fill="10" visible="no" active="yes"/>
 <layer number="44" name="Drills" color="7" fill="1" visible="no" active="yes"/>
 <layer number="45" name="Holes" color="7" fill="1" visible="no" active="yes"/>
-<layer number="46" name="Milling" color="3" fill="1" visible="yes" active="yes"/>
-<layer number="47" name="Measures" color="7" fill="1" visible="yes" active="yes"/>
-<layer number="48" name="Document" color="7" fill="1" visible="yes" active="yes"/>
-<layer number="49" name="Reference" color="7" fill="1" visible="yes" active="yes"/>
+<layer number="46" name="Milling" color="3" fill="1" visible="no" active="yes"/>
+<layer number="47" name="Measures" color="7" fill="1" visible="no" active="yes"/>
+<layer number="48" name="Document" color="7" fill="1" visible="no" active="yes"/>
+<layer number="49" name="Reference" color="7" fill="1" visible="no" active="yes"/>
 <layer number="50" name="dxf" color="12" fill="1" visible="no" active="no"/>
 <layer number="51" name="tDocu" color="7" fill="1" visible="yes" active="yes"/>
@@
 <autorouter>
 <pass name="Default">
-<param name="RoutingGrid" value="8mil"/>
+<param name="RoutingGrid" value="14mil"/>
 <param name="tpViaShape" value="round"/>
 <param name="PrefDir.1" value="|"/>
@@
 <element name="C2" library="rcl" package="C1206" value="22pF" x="34.29" y="41.91" smashed="yes">
 <attribute name="NAME" x="33.02" y="43.18" size="1.27" layer="25"/>
-<attribute name="VALUE" x="27.305" y="41.275" size="1.27" layer="27"/>
+<attribute name="VALUE" x="32.7025" y="43.18" size="1.27" layer="27"/>
 </element>
 <element name="C8" library="rcl" package="C1206" value="22pF" x="34.29" y="36.83" smashed="yes">
 <attribute name="NAME" x="33.02" y="38.1" size="1.27" layer="25"/>
-<attribute name="VALUE" x="20.955" y="34.925" size="1.27" layer="27"/>
+<attribute name="VALUE" x="31.75" y="34.29" size="1.27" layer="27"/>
 </element>
 <element name="R13" library="rcl" package="R1206" value="1M" x="43.18" y="39.37" smashed="yes" rot="R270">
@@
 <attribute name="VALUE" x="50.8635" y="25.3365" size="1.27" layer="27" rot="R90"/>
 </element>
-<element name="C3" library="rcl" package="C1206" value="100nF" x="54.9275" y="49.53" smashed="yes" rot="R180">
-<attribute name="NAME" x="56.1975" y="48.26" size="1.27" layer="25" rot="R180"/>
-<attribute name="VALUE" x="57.4675" y="52.07" size="1.27" layer="27" rot="R180"/>
+<element name="C3" library="rcl" package="C1206" value="100nF" x="52.3875" y="48.895" smashed="yes" rot="R180">
+<attribute name="NAME" x="53.6575" y="47.625" size="1.27" layer="25" rot="R180"/>
+<attribute name="VALUE" x="54.9275" y="51.435" size="1.27" layer="27" rot="R180"/>
 </element>
 <element name="X3" library="lpatiny" package="NX6035" value="16MHz" x="39.37" y="39.37" smashed="yes" rot="R90">
@@
 <element name="RL2" library="rcl" package="R0805" value="1K" x="17.78" y="12.7" rot="R180"/>
 <element name="J7" library="lpatiny" package="2-PIN-5.08S" value="22--02" x="25.4" y="6.35" rot="R180"/>
-<element name="LED13" library="adafruit" package="CHIPLED_1206" value="RED" x="17.78" y="44.45" rot="R90"/>
+<element name="LED13" library="adafruit" package="CHIPLED_1206" value="RED" x="17.78" y="44.45" smashed="yes" rot="R90">
+<attribute name="NAME" x="19.05" y="43.18" size="1.27" layer="25" rot="R180"/>
+<attribute name="VALUE" x="19.05" y="46.99" size="1.27" layer="27" rot="R180"/>
+</element>
 <element name="LED14" library="adafruit" package="CHIPLED_1206" value="GREEN" x="17.78" y="46.99" rot="R90"/>
 <element name="IC2" library="analog-devices" package="SO8" value="AD8223" x="46.99" y="16.51">
@@
 <wire x1="58.8137" y1="45.085" x2="60.41" y2="42.57" width="0" layer="19" extent="1-16"/>
 <wire x1="55.41" y1="45.17" x2="58.8137" y2="45.085" width="0" layer="19" extent="1-16"/>
-<wire x1="56.3275" y1="49.53" x2="55.41" y2="45.17" width="0" layer="19" extent="1-1"/>
 <wire x1="48.81" y1="40.97" x2="55.41" y2="45.17" width="0" layer="19" extent="1-1"/>
 <wire x1="50.61" y1="33.57" x2="48.81" y2="40.97" width="0" layer="19" extent="1-1"/>
 <wire x1="54.61" y1="6.35" x2="56.01" y2="15.24" width="0" layer="19" extent="1-1"/>
 <wire x1="76.2" y1="6.35" x2="62.865" y2="20.32" width="0" layer="19" extent="1-16"/>
+<wire x1="53.7875" y1="48.895" x2="55.41" y2="48.895" width="0.4064" layer="1"/>
+<wire x1="55.41" y1="48.895" x2="55.41" y2="45.17" width="0.4064" layer="1"/>
 </signal>
 <signal name="SCK">
@@
 <contactref element="U$4" pad="3"/>
 <contactref element="R31" pad="1"/>
-<wire x1="35.69" y1="50.165" x2="57.01" y2="45.17" width="0" layer="19" extent="1-1"/>
 <wire x1="25.08" y1="44.45" x2="35.69" y2="50.165" width="0" layer="19" extent="1-1"/>
+<wire x1="35.69" y1="50.165" x2="46.99" y2="50.165" width="0.4064" layer="1"/>
+<wire x1="46.99" y1="50.165" x2="46.99" y2="52.07" width="0.4064" layer="1"/>
+<wire x1="46.99" y1="52.07" x2="57.01" y2="52.07" width="0.4064" layer="1"/>
+<wire x1="57.01" y1="52.07" x2="57.01" y2="45.17" width="0.4064" layer="1"/>
 </signal>
 <signal name="RD+">
@@
 <contactref element="U$4" pad="4"/>
 <contactref element="R24" pad="1"/>
-<wire x1="35.69" y1="46.99" x2="56.21" y2="45.17" width="0" layer="19" extent="1-1"/>
+<wire x1="35.69" y1="46.99" x2="48.26" y2="46.99" width="0.4064" layer="1"/>
+<wire x1="48.26" y1="46.99" x2="48.26" y2="50.8" width="0.4064" layer="1"/>
+<wire x1="48.26" y1="50.8" x2="56.21" y2="50.8" width="0.4064" layer="1"/>
+<wire x1="56.21" y1="50.8" x2="56.21" y2="45.17" width="0.4064" layer="1"/>
 <wire x1="25.08" y1="46.99" x2="35.69" y2="46.99" width="0" layer="19" extent="1-1"/>
 </signal>
@@
 <contactref element="X4" pad="2"/>
 <contactref element="R31" pad="2"/>
-<wire x1="8.08" y1="49.06" x2="32.89" y2="50.165" width="0" layer="19" extent="1-1"/>
+<wire x1="8.08" y1="49.06" x2="29.21" y2="49.06" width="0.4064" layer="1"/>
+<wire x1="29.21" y1="49.06" x2="29.21" y2="49.53" width="0.4064" layer="1"/>
+<wire x1="29.21" y1="49.53" x2="32.89" y2="49.53" width="0.4064" layer="1"/>
+<wire x1="32.89" y1="49.53" x2="32.89" y2="50.165" width="0.4064" layer="1"/>
 </signal>
 <signal name="D+USB">
 <contactref element="X4" pad="3"/>
 <contactref element="R24" pad="2"/>
-<wire x1="8.08" y1="48.26" x2="32.89" y2="46.99" width="0" layer="19" extent="1-1"/>
+<wire x1="8.08" y1="48.26" x2="32.89" y2="48.26" width="0.4064" layer="1"/>
+<wire x1="32.89" y1="48.26" x2="32.89" y2="46.99" width="0.4064" layer="1"/>
 </signal>
 <signal name="N$8">
@@
 <contactref element="U$4" pad="6"/>
 <contactref element="C3" pad="2"/>
-<wire x1="54.61" y1="45.17" x2="53.5275" y2="49.53" width="0" layer="19" extent="1-1"/>
+<wire x1="50.9875" y1="48.895" x2="50.8" y2="48.26" width="0.4064" layer="1"/>
+<wire x1="50.8" y1="48.26" x2="50.8" y2="46.99" width="0.4064" layer="1"/>
+<wire x1="50.8" y1="46.99" x2="54.61" y2="46.99" width="0.4064" layer="1"/>
+<wire x1="54.61" y1="46.99" x2="54.61" y2="45.17" width="0.4064" layer="1"/>
 </signal>
 <signal name="D12*">
