File: PCB/anemometer/v2/anemo2.sch (EAGLE design)
At the start: 63 parts, among them IC1 AD620R, IC2 AD620R, IC3 AD620R, IC4 AD620R, IC6 TL072D, J1 RJ12STRAIGHT-I2C, T1 BC846, T2 BC846, T3 BC846, T4 BC846

Commit message: added version 2 that was sent to factory
Parts:
- removed IC6: TL072D, linear:TL072D
- removed PT100_1, PT100_2, PT100_3, PT100_4, PT1K_1, PT1K_2, PT1K_3, PT1K_4: 90.9, resistor:R-EU_M1206
- removed U$1: MCP3424(SO14), mcp3424:MCP3424(SO14)
- added IC5: TL072P, linear:TL072P
- added U1: (no value), SparkFun-DigitalIC:TXB0104PWRSOIC14
- added X1, X2, X3, X4: 14867, con-4ucon:14867
- DIV1, DIV3, DIV5, DIV7: value 20k -> 10
- DIV2, DIV4, DIV6, DIV8: value 10k -> 10
- IC1, IC2, IC3, IC4: value AD620R -> AD620N; device analog-devices:AD620R -> analog-devices:AD620N
- RT_1, RT_2, RT_3, RT_4: value 90.9 -> 82.5
Connections:
- net 5V: no longer U$1.VDD
- net ADR0: no longer U$1.ADR0
- net ADR1: now also U1.B4; no longer U$1.ADR1
- net GND: now also U1.A1, U1.A3, U1.A4, U1.B2, U1.VCCB, X1.1, X1.4, X2.1, X2.4, X3.1, X3.4, X4.1, X4.4; no longer IC6P.V-, PT100_1.1, PT100_2.1, PT100_3.1, PT100_4.1, PT1K_1.1, PT1K_2.1, PT1K_3.1, PT1K_4.1, U$1.CH1-, U$1.CH2-, U$1.CH3-, U$1.CH4-, U$1.VSS
- net IN-1: now also X1.3; no longer PT100_1.2
- net IN-2: now also X2.3; no longer PT100_2.2
- net IN-3: now also X3.3; no longer PT100_3.2
- net IN-4: now also X4.3; no longer PT100_4.2
- net N$10: now also IC5A.+IN; no longer IC6A.+IN
- net N$23: now also X1.2; no longer PT1K_1.2
- net N$25: now also X2.2; no longer PT1K_2.2
- net N$27: now also X3.2; no longer PT1K_3.2
- net N$29: now also X4.2; no longer PT1K_4.2
- net REF: now also IC5A.-IN, IC5A.OUT; no longer IC6A.-IN, IC6A.OUT
- net SCL: now also U1.OE; no longer U$1.SCL
- net SDA: now also U1.GND; no longer U$1.SDA
- net SIG1: now also U1.VCCA; no longer U$1.CH1+
- net SIG2: now also U1.A2; no longer U$1.CH2+
- net SIG3: now also U1.B3; no longer U$1.CH3+
- net SIG4: now also U1.B1; no longer U$1.CH4+
- net VCC: no longer IC6P.V+
