File: PCB/anemometer/v3.1/routed_anemo3.sch (EAGLE design)
At the start: 66 parts, among them IC1 AD8223, IC2 AD8223, IC3 AD8223, IC4 AD8223, IC6 TL072D, J1 RJ12STRAIGHT-I2C, J2 RJ12STRAIGHT-I2C, T1 BC846, T2 BC846, T3 BC846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

Commit message: added version 2 that was sent to factory
Changed lines of the file:
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@@
 <pinref part="U$1" gate="G$1" pin="VDD"/>
 <wire x1="-12.7" y1="-73.66" x2="-20.32" y2="-73.66" width="0.1524" layer="91"/>
-<label x="-17.78" y="-71.12" size="1.778" layer="95"/>
+<label x="-17.78" y="-73.66" size="1.778" layer="95"/>
 </segment>
 <segment>
