File: PCB/IntegratedBertha/v1.1/integratedBertha.sch (EAGLE design)
At the start: 96 parts, among them CON1 SPI, IC1 REG1117, IC2 AD8223, J1 RJ12, J2 RJ12, J3 RJ12, J4 RJ12, J5 RJ12, J7 22--02, Q1 BSP75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

Commit message: added RF filter capacitances. autorouter works still 100percent
Parts:
- added C13: 4.7uF, rcl:C-EUC1206
- added C14, C15: 100nF, rcl:C-EUC1206
- added R19, R20: 49.9, resistor:R-EU_R1206
- U$4: value ATMEGA32U4-AU -> ATMEGA32U4
Connections:
- new net N$31: R20.2, X1-2.S
- new net N$37: R19.2, X1-3.S
- net +5V: now also C4.2; no longer C4.1
- net DIFF+: now also C13.1, C14.2, R19.1; no longer X1-3.S
- net DIFF-: now also C13.2, C15.1, R20.1; no longer X1-2.S
- net GND: now also C14.1, C15.2, C4.1; no longer C4.2
Other:
- moved on the sheet: C4, C6, IC2, R2, R9, X1-1, X1-2, X1-3, X1-4
