File: PCB/IntegratedBertha/v1_1b/integratedBertha.brd (EAGLE design)
At the start: 108.1 x 84.6 mm, 100 parts, among them CON1 SPI, IC1 REG1117, IC2 AD8223, J7 22--02, Q1 BSP75, Q2 BSP75, Q4 BSP75, Q5 BSP75, Q6 BSP75, Q7 IRF3704S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

Commit message: also in v1_1b
Parts:
- C16: value 100uF -> 100nF
Changed lines of the file:
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@@
 </element>
 <element name="U$2" library="lpatiny" package="STAR" value="STARGND" x="22.8854" y="20.6248" rot="MR0"/>
-<element name="C16" library="rcl" package="C1206" value="100uF" x="50.2158" y="27.7368" smashed="yes" rot="R90">
+<element name="C16" library="rcl" package="C1206" value="100nF" x="50.2158" y="27.7368" smashed="yes" rot="R90">
 <attribute name="VALUE" x="49.5808" y="25.1968" size="1.016" layer="27" rot="R90"/>
 </element>
