File: PCB/IntegratedBertha/v1_1b/integratedBertha.sch (EAGLE design)
At the start: 100 parts, among them CON1 SPI, IC1 REG1117, IC2 AD8223, J7 22--02, Q1 BSP75, Q2 BSP75, Q4 BSP75, Q5 BSP75, Q6 BSP75, Q7 IRF3704S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

Commit message: also in v1_1b
Parts:
- C16: value 100uF -> 100nF
Changed lines of the file:
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@@
 <part name="AGND3" library="supply2" deviceset="AGND" device="" value="AGND"/>
 <part name="AGND4" library="supply2" deviceset="AGND" device="" value="AGND"/>
-<part name="C16" library="rcl" deviceset="C-EU" device="C1206" value="100uF"/>
+<part name="C16" library="rcl" deviceset="C-EU" device="C1206" value="100nF"/>
 <part name="L1" library="rcl" deviceset="L-US" device="L2012C" value="10uH"/>
 <part name="AGND6" library="supply2" deviceset="AGND" device="" value="AGND"/>
