File: Wiegand/Door locking pcb v1.0/Door locking pcb.brd (EAGLE design)
At the start: 108.1 x 61.7 mm, 52 parts, among them CON1 SPI, J1 22--02, J7 22--02, Q3 BSP75, X3 16MHz, X4 MINI-USB

Commit message: corrected errors in wiedgand
Parts:
- removed LED13: RED, adafruit:CHIPLED_1206
- removed LED14: GREEN, adafruit:CHIPLED_1206
- removed RL1, RL7: 1K, rcl:R0805
- added Q1: BSP75, infineon:PG-SOT-223
- moved J1 3.81 mm to (85.1, 8.89), turned to 0 degrees
- moved Q3 2.54 mm to (99.1, 12.7), turned to 0 degrees
Connections:
- removed net N$14: LED14.A, RL7.2
- removed net N$8: LED13.A, RL1.2
- new net N$1: PIN3.P$3, PIN4.P$3, Q1.2
- net CS: now also Q1.1; no longer PIN3.P$3, PIN4.P$3
- net GND: now also Q1.3; no longer LED13.C, LED14.C
- net RD+: no longer RL7.1
- net RD-: no longer RL1.1
Routing:
- net N$1: track 0.00 -> 25.1 mm
- net RD-: track 67.9 -> 43.4 mm
- net CS: track 43.0 -> 31.3 mm
- net RESET: track 57.2 -> 67.5 mm
- net GND: track 445.9 -> 435.9 mm, vias 3 -> 2
- net +12V: track 205.1 -> 196.2 mm
- net RD+: track 41.7 -> 36.2 mm
- net N$2: track 24.3 -> 20.1 mm, vias 2 -> 0
- net N$8: track 3.65 -> 0.00 mm
- net N$14: track 3.65 -> 0.00 mm
- net D12*: track 58.9 -> 61.3 mm, vias 0 -> 2
Other:
- board text added: "BLA"
- board text added: "BLU"
- board text added: "GRE"
- board text added: "RED"
- board text added: "WHI"
- board text added: "YEL"
- board text removed: "Buzzer"
- board text removed: "D0"
- board text removed: "D1"
