File: PCB/Control board pH/v1.0/ControlBoardpH.brd (EAGLE design)
At the start: 108.1 x 84.6 mm, 92 parts, among them CON1 SPI, IC1 REG1117, J1 RJ12, J2 RJ12, J3 RJ12, J4 RJ12, J5 RJ12, J7 22--02, Q1 BSP75, Q2 BSP75, Q4 BSP75, Q5 BSP75, Q6 BSP75, Q7 IRF3704S, X2 22-23-20315.08S, X3 16MHz, X4 MINI-USB, X5 22-23-20315.08S, X6 87758-4016

Commit message: ph meter independant
Parts:
- removed L_AVCC: 100mH, resistor:R1206
- added C13: 4.7uF, rcl:C1206
- added C14, C15, C22: 100nF, rcl:C1206
- added C19, C21: 100n, rcl:C1206
- added C20: 0.000010, rcl:C1206
- added C23: 10uF, rcl:C1206
- added I/O_PWM: I2C 1, lpatiny:RJ12-STRAIGHT
- added IC2: AD8223, analog-devices:SO8
- added IC3: TL084D, linear:SO14
- added J6: RJ12STRAIGHT, lpatiny:RJ12-STRAIGHT
- added J8: RJ12STRAIGHT-I2C, lpatiny:RJ12-STRAIGHT-I2C
- added K1, K2: JS-M1-9V-5, relay:JS-M
- added LED0, LED15, LED16: (no value), SparkFun:LED-1206
- added LED13: RED, adafruit:CHIPLED_1206
- added LED14: GREEN, adafruit:CHIPLED_1206
- added Q3: BSP75, infineon:PG-SOT-223
- added R13: 1M, rcl:R1206
- added R19, R20: 49.9, resistor:R1206
- added R2: 300, resistor:R1206
- added R22: 1k, resistor:R1206
- added R23: 124k, resistor:R1206
- added R26, R30, R36, R42: 100k, resistor:R1206
- added R37: 2.2k, resistor:R1206
- added R38: 110k, resistor:R1206
- added R40: 750, resistor:R1206
- added R41: 240k, resistor:R1206
- added R43, RL0, RL9: 1K, resistor:M1206
- added R44: 10K, LCD:ECP10S
- added R9: 100, resistor:R1206
- added RL1, RL7: 1K, rcl:R0805
- added U$10: LCD-16PINS, lcd-hd44780:LCD-16PINS
- added U$12: LCD-14PINS, lcd-hd44780:LCD-14PINS
- added U$4: ATMEGA32U4, adafruit:TQFP44
- added U$5: VERTICAL-JACK, phMeter:VERTICAL-JACK
- added U$9: MCP3425, phMeter:SOT-23-6
- added V1, V2, V3, V4, V5: (no value), pinhead:1X01
- added X1: 22-23-20415.08S, lpatiny:4-PIN-5.08S
- added X7: 22-23-20315.08S, lpatiny:3-PIN-5.08S
- C16: value 1uF -> 100n
- C17: value 100nF -> 100n
- C18: value 100nF -> 22000n
- C2, C8: value 10pF -> 22pF
- C3, C4: value 1uF -> 100nF
- C6: value 1uF -> 330nF
- LED10, LED4: value (none) -> RED
- LED3: value REDx3 -> RED
- R27: value 1Kx3 -> 1K
- R3: value 1k -> 10k
- RL3, RL4: value (none) -> 1K
- U$2: value AT90USB1286 -> BNC-VERTICAL; device lpatiny:TQFP64 -> phMeter:BNC-VERTICAL
- U$3: value SZ05-ZIGBEETHROUGHHOLE -> SZ05-ZIGBEE; device lpatiny:SZ05-ZIGBEE4 -> lpatiny:SZ05-ZIGBEE
- X6: value 87758-4016 -> 22-23-20315.08S; device con-molex:87758-4016 -> lpatiny:3-PIN-5.08S
- moved X6 97.0 mm to (24.1, -86.4), turned to 0 degrees
- moved C17 89.8 mm to (21.0, -42.5)
- moved C18 89.1 mm to (5.71, -42.5), turned to 0 degrees
- moved C16 87.6 mm to (14.6, -42.5), turned to 0 degrees
- moved U$2 84.9 mm to (-6.35, -23.5), turned to 0 degrees
- moved U$1 46.5 mm to (55.9, 47.0), flipped to the bottom
- moved C3 42.7 mm to (52.4, 48.9), flipped to the top, turned to 180 degrees
- moved R16 39.8 mm to (63.5, 48.3), turned to 180 degrees
- moved X5 35.7 mm to (92.7, 6.35), turned to 0 degrees
- moved R17 34.3 mm to (63.5, 45.7)
- moved X2 32.7 mm to (71.1, 6.35), turned to 0 degrees
- moved LED1 31.2 mm to (63.5, 26.7), turned to 0 degrees
- moved C4 29.7 mm to (47.0, 26.9), turned to 180 degrees
- moved RL5 29.4 mm to (67.3, 26.7), turned to 270 degrees
- moved RESET1 28.6 mm to (54.6, 26.7), flipped to the bottom, turned to 180 degrees
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Connections:
- net USBC_N renamed D-USB
- net USBC_P renamed D+USB
- removed net A6: U$2.60
- removed net A7: U$2.61
- removed net TFT-CS: U$2.33, X6.11
- removed net TFT-DB0: U$2.35, X6.40
- removed net TFT-DB1: U$2.36, X6.38
- removed net TFT-DB10: U$2.49, X6.23
- removed net TFT-DB11: U$2.48, X6.21
- removed net TFT-DB12: U$2.47, X6.19
- removed net TFT-DB13: U$2.46, X6.17
- removed net TFT-DB14: U$2.45, X6.15
- removed net TFT-DB15: U$2.44, X6.13
- removed net TFT-DB2: U$2.37, X6.36
- removed net TFT-DB3: U$2.38, X6.34
- removed net TFT-DB4: U$2.39, X6.32
- removed net TFT-DB5: U$2.40, X6.30
- removed net TFT-DB6: U$2.41, X6.28
- removed net TFT-DB7: U$2.42, X6.26
- removed net TFT-DB8: U$2.51, X6.27
- removed net TFT-DB9: U$2.50, X6.25
- removed net TFT-RESET: U$2.34, X6.7
- removed net TFT-RS: U$2.18, X6.33
- removed net TFT-WR: U$2.19
- removed net TST-WR: X6.31
- removed net USB_N: R31.1, U$2.4
- removed net USB_P: R24.1, U$2.5
- new net DIFF+: C13.1, C14.2, IC2.3, R19.1
- new net DIFF-: C13.2, C15.1, IC2.2, R20.1
- new net I/O: I/O_PWM.I/O, IC3.8, J6.I/O, Q3.1, R40.2, U$9.VIN+, V4.1
- new net N$15: IC2.8, R2.1
- new net N$16: C3.2, U$4.6
- new net N$31: R20.2, X1.2
- new net N$37: R19.2, X1.3
- new net N$38: J6.PWM, R22.2
- new net N$40: IC2.6, R9.1
- new net N$41: IC3.2, R23.1, R26.2
- new net N$42: C8.2, R13.2, U$4.17, X3.P$2
- new net N$43: C17.2, IC3.5, R30.1, R36.2
- new net N$44: IC3.1, R23.2, R37.1, V2.1
- new net N$45: C18.2, IC3.10, R37.2, V3.1
- new net N$46: IC3.9, R38.2, R40.1
- new net N$47: IC3.13, IC3.14, U$9.VIN-, V5.1
- new net N$48: C21.2, IC3.12, R41.1, R42.2
- new net N$49: K2.1, LED15.C, Q3.2
- new net N$50: LED0.A, RL0.1
- new net N$51: LED15.A, RL9.1
- new net N$52: LED16.A, R43.1
- new net N$53: K2.NO, X6.1
- new net N$54: K1.NO, X7.1
- new net N$55: K1.NC, X7.3
- new net N$56: K2.NC, X6.3
- new net N$57: K2.C, X6.2
- new net N$58: R44.S, U$12.3
- new net POWER1: K1.C, X7.2
- new net PWM: I/O_PWM.PWM, K1.1, LED0.C
- new net RA0: U$12.4
- new net RA1: U$12.6
- new net RA2: U$12.11
- new net RC0: U$12.12
- new net RC1: U$12.13
- new net RC2: U$12.14
- new net RD+: R24.1, RL7.1, U$4.4
- new net RD-: R31.1, RL1.1, U$4.3
- new net XTAL1: C2.2, R13.1, U$4.16, X3.P$1
- net +5V: now also C16.1, C19.2, C20.2, C22.1, C23.1, C4.2, I/O_PWM.+5V, IC2.7, IC3.4, J6.+5V, J8.+5V, K1.2, K2.2, R22.1, R30.2, R41.2, R43.2, R44.A, RL0.2, RL9.2, U$12.2, U$9.VDD, X1.1
- net +5V/1: now also U$4.14, U$4.2, U$4.24, U$4.34, U$4.44; no longer C17.1, C18.1, C4.1, L_AVCC.1, U$2.21, U$2.52, X6.3, X6.37
- net 3.3V: no longer X6.29
- net A0: now also U$4.36; no longer U$2.54
- net A1: now also R33.1, U$4.37; no longer R.1, U$2.55
- net A2: now also U$4.38; no longer U$2.56
- net A3: now also R.1, U$4.39; no longer R33.1, U$2.57
- net A4: now also U$4.40; no longer U$2.58
- net A5: now also U$4.41; no longer R35.1, U$2.59
- net AREF: now also U$4.42; no longer U$2.62
- net CS: now also U$4.25; no longer U$2.29
- net D10*: now also Q2.1, U$4.30; no longer Q4.1, U$2.16
- net D11*: now also Q6.1, U$4.12; no longer Q5.1, U$2.17
- net D12*: now also C6.1, R9.2, U$4.26; no longer U$2.31
- net D13*: now also U$4.32; no longer U$2.9
- net D5*: now also Q5.1, U$4.31; no longer Q6.1, U$2.2
- net D6*: now also Q1.1, U$4.27; no longer U$2.32
- net D7*: now also U$4.1; no longer U$2.1
- net D8*: now also R35.1, U$4.28; no longer Q1.1, U$2.14
- net D9*: now also Q4.1, U$4.29; no longer Q2.1, U$2.15
- net GND: now also C14.1, C15.2, C16.2, C17.1, C18.1, C19.1, C20.1, C21.1, C22.2, C23.2, C4.1, I/O_PWM.GND2, IC2.4, IC2.5, IC3.11, J6.GND1, J6.GND2, J8.GND1, J8.GND2, LED13.C, LED14.C, LED16.C, Q3.3, R36.1, R38.1, R42.1, R44.E, U$12.1, U$12.10, U$12.5, U$12.7, U$12.8, U$12.9, U$3.SGND, U$4.15, U$4.23, U$4.35, U$4.43, U$4.5, U$5.P$1, U$5.P$2, U$9.VSS, X1.4; no longer C16.1, C17.2, C18.2, C4.2, U$2.22, U$2.53, U$2.6, U$2.63, U$3.SND, X6.39
- net GND1: now also U$3.RNU; no longer U$3.RUN
- net HWB: now also U$4.33; no longer U$2.43
- net MISO: now also U$4.11; no longer U$2.13
- net MOSI: now also U$4.10; no longer U$2.12
- net N$13: now also IC2.1, R2.2; no longer C6.1, L_AVCC.2, U$2.64
- net N$14: now also LED14.A, RL7.2; no longer C2.2, U$2.24, X3.P$2
- net N$2: now also IC3.6, IC3.7, R26.1, U$2.G, V1.1
- net N$39: now also IC3.3, U$2.S; no longer C8.2, U$2.23, X3.P$1
- net N$8: now also LED13.A, RL1.2; no longer C3.2, U$2.7
- net RESET: now also U$4.13; no longer U$2.20
- net RX: now also U$4.20; no longer U$2.27
- net RXLED: now also U$4.8; no longer U$2.10
- net SCK: now also U$4.9; no longer U$2.11
- net SCL: now also J8.SCL, U$4.18, U$9.SCL; no longer U$2.25
- net SDA: now also J8.SDA, U$4.19, U$9.SDA; no longer U$2.26
- net TX: now also U$4.21; no longer U$2.28
- net TXLED: now also U$4.22; no longer U$2.30
- net VUSB: now also U$4.7; no longer C16.2, U$2.3, U$2.8
Routing:
- net GND: track 686.1 -> 409.8 mm, vias 14 -> 0
- net +5V/1: track 171.8 -> 0.00 mm, vias 3 -> 0
- net 3.3V: track 141.8 -> 0.00 mm, vias 5 -> 0
- net SDA: track 122.7 -> 26.4 mm, vias 1 -> 0
- net FMOSI: track 91.6 -> 0.00 mm, vias 1 -> 0
- net A5: track 89.0 -> 0.00 mm, vias 2 -> 0
- net D7*: track 82.1 -> 0.00 mm, vias 2 -> 0
- net SCL: track 97.6 -> 22.2 mm, vias 3 -> 0
- net ISP+5V: track 74.8 -> 0.00 mm, vias 1 -> 0
- net VUSB: track 74.7 -> 0.00 mm, vias 4 -> 0
- net RESET: track 72.3 -> 0.00 mm, vias 4 -> 0
- net +5V: track 432.3 -> 361.2 mm, vias 3 -> 1
- net TFT-DB7: track 67.3 -> 0.00 mm, vias 2 -> 0
- net MOSI: track 61.5 -> 0.00 mm, vias 2 -> 0
- net TFT-DB6: track 61.1 -> 0.00 mm, vias 1 -> 0
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- removed copper zone on layer 16, net GND
Other:
- board text added: "+"
- board text added: "-"
- board text added: "Weight"
- board text removed: "+5V"
- board text removed: "CS"
- board text removed: "DB0"
- board text removed: "DB1"
- board text removed: "DB10"
- board text removed: "DB11"
- board text removed: "DB12"
- board text removed: "DB13"
- board text removed: "DB14"
- board text removed: "DB15"
- board text removed: "DB2"
- board text removed: "DB3"
- board text removed: "DB4"
- board text removed: "DB5"
- board text removed: "DB6"
- board text removed: "DB7"
- board text removed: "DB8"
- board text removed: "DB9"
- board text removed: "LEd"
- board text removed: "RD"
- board text removed: "RS"
- board text removed: "RSET"
- board text removed: "Screen"
- board text removed: "WR"
