File: PCB/Control board pH/v1.0/ControlBoardpH.sch (EAGLE design)
At the start: 92 parts, among them CON1 SPI, IC1 REG1117, J1 RJ12, J2 RJ12, J3 RJ12, J4 RJ12, J5 RJ12, J7 22--02, Q1 BSP75, Q2 BSP75, Q4 BSP75, Q5 BSP75, Q6 BSP75, Q7 IRF3704S, X2 22-23-20315.08S, X3 16MHz, X4 MINI-USB, X5 22-23-20315.08S, X6 87758-4016

Commit message: ph meter independant
Parts:
- removed L_AVCC: 100mH, resistor:R-EU_R1206
- added C13: 4.7uF, rcl:C-EUC1206
- added C14, C15, C22: 100nF, rcl:C-EUC1206
- added C19, C21: 100n, rcl:C-EUC1206
- added C20: 0.000010, rcl:C-EUC1206
- added C23: 10uF, rcl:C-EUC1206
- added I/O_PWM: I2C 1, lpatiny:RJ12STRAIGHT
- added IC2: AD8223, analog-devices:AD620R
- added IC3: TL084D, linear:TL084D
- added J6: RJ12STRAIGHT, lpatiny:RJ12STRAIGHT
- added J8: RJ12STRAIGHT-I2C, lpatiny:RJ12STRAIGHT-I2C
- added K1, K2: JS-M1-9V-5, relay:JS-M1-9V-5
- added LED0, LED15, LED16: (no value), SparkFun:LED1206
- added LED13: RED, adafruit:LEDCHIPLED_1206
- added LED14: GREEN, adafruit:LEDCHIPLED_1206
- added Q3: BSP75, infineon:BSP613P
- added R13: 1M, rcl:R-EU_R1206
- added R19, R20: 49.9, resistor:R-EU_R1206
- added R2: 300, resistor:R-EU_R1206
- added R22: 1k, resistor:R-EU_R1206
- added R23: 124k, resistor:R-EU_R1206
- added R26, R30, R36, R42: 100k, resistor:R-EU_R1206
- added R37: 2.2k, resistor:R-EU_R1206
- added R38: 110k, resistor:R-EU_R1206
- added R40: 750, resistor:R-EU_R1206
- added R41: 240k, resistor:R-EU_R1206
- added R43, RL0, RL9: 1K, resistor:R-EU_M1206
- added R44: 10K, LCD:TRIM_US-ECP10S
- added R9: 100, resistor:R-EU_R1206
- added RL1, RL7: 1K, rcl:R-EU_R0805
- added U$10: LCD-16PINS, lcd-hd44780:LCD-16PINS
- added U$12: LCD-14PINS, lcd-hd44780:LCD-14PINS
- added U$4: ATMEGA32U4, adafruit:ATMEGA32U4-AU
- added U$5: VERTICAL-JACK, phMeter:VERTICAL-JACK
- added U$9: MCP3425, phMeter:MCP3425
- added V1, V2, V3, V4, V5: (no value), pinhead:PINHD-1X1
- added X1: 22-23-20415.08S, lpatiny:22-23-20415.08S
- added X7: 22-23-20315.08S, lpatiny:22-23-20315.08S
- C16: value 1uF -> 100n
- C17: value 100nF -> 100n
- C18: value 100nF -> 22000n
- C2, C8: value 10pF -> 22pF
- C3, C4: value 1uF -> 100nF
- C6: value 1uF -> 330nF
- LED10, LED4: value (none) -> RED
- LED3: value REDx3 -> RED
- R27: value 1Kx3 -> 1K
- R3: value 1k -> 10k
- RL3, RL4: value (none) -> 1K
- U$2: value AT90USB1286 -> BNC-VERTICAL; device lpatiny:AT90USB1286TQFP64 -> phMeter:BNC-VERTICAL
- U$3: value SZ05-ZIGBEETHROUGHHOLE -> SZ05-ZIGBEE; device lpatiny:SZ05-ZIGBEETHROUGHHOLE -> lpatiny:SZ05-ZIGBEE
- X6: value 87758-4016 -> 22-23-20315.08S; device con-molex:87758-4016 -> lpatiny:22-23-20315.08S
Connections:
- net USBC_N renamed D-USB
- net USBC_P renamed D+USB
- removed net A6: U$2.PF1(ADC1)
- removed net A7: U$2.PF0(ADC0)
- removed net TFT-CS: U$2.PE0, X6-11.S
- removed net TFT-DB0: U$2.PC0, X6-40.S
- removed net TFT-DB1: U$2.PC1, X6-38.S
- removed net TFT-DB10: U$2.PA2, X6-23.S
- removed net TFT-DB11: U$2.PA3, X6-21.S
- removed net TFT-DB12: U$2.PA4, X6-19.S
- removed net TFT-DB13: U$2.PA5, X6-17.S
- removed net TFT-DB14: U$2.PA6, X6-15.S
- removed net TFT-DB15: U$2.PA7, X6-13.S
- removed net TFT-DB2: U$2.PC2, X6-36.S
- removed net TFT-DB3: U$2.PC3(T3), X6-34.S
- removed net TFT-DB4: U$2.PC4(OC3C), X6-32.S
- removed net TFT-DB5: U$2.PC5(OC3B), X6-30.S
- removed net TFT-DB6: U$2.PC6(OC3A), X6-28.S
- removed net TFT-DB7: U$2.PC7(IC3), X6-26.S
- removed net TFT-DB8: U$2.PA0, X6-27.S
- removed net TFT-DB9: U$2.PA1, X6-25.S
- removed net TFT-RESET: U$2.PE1, X6-7.S
- removed net TFT-RS: U$2.PE4(TOSC1/INT4), X6-33.S
- removed net TFT-WR: U$2.PE5(TOSC2/INT5)
- removed net TST-WR: X6-31.S
- removed net USB_N: R31.1, U$2.D-
- removed net USB_P: R24.1, U$2.D+
- new net DIFF+: C13.1, C14.2, IC2.+, R19.1
- new net DIFF-: C13.2, C15.1, IC2.-, R20.1
- new net I/O: I/O_PWM.3, IC3C.OUT, J6.3, Q3.G, R40.2, U$9.VIN+, V4.1
- new net N$15: IC2.RG@2, R2.1
- new net N$16: C3.2, U$4.UCAP
- new net N$31: R20.2, X1-2.S
- new net N$37: R19.2, X1-3.S
- new net N$38: J6.2, R22.2
- new net N$40: IC2.OUT, R9.1
- new net N$41: IC3A.-IN, R23.1, R26.2
- new net N$42: C8.2, R13.2, U$4.XTAL1, X3.P$2
- new net N$43: C17.2, IC3B.+IN, R30.1, R36.2
- new net N$44: IC3A.OUT, R23.2, R37.1, V2.1
- new net N$45: C18.2, IC3C.+IN, R37.2, V3.1
- new net N$46: IC3C.-IN, R38.2, R40.1
- new net N$47: IC3D.-IN, IC3D.OUT, U$9.VIN-, V5.1
- new net N$48: C21.2, IC3D.+IN, R41.1, R42.2
- new net N$49: K21.1, LED15.C, Q3.D@1
- new net N$50: LED0.A, RL0.1
- new net N$51: LED15.A, RL9.1
- new net N$52: LED16.A, R43.1
- new net N$53: K22.S, X6-1.S
- new net N$54: K12.S, X7-1.S
- new net N$55: K12.O, X7-3.S
- new net N$56: K22.O, X6-3.S
- new net N$57: K22.P, X6-2.S
- new net N$58: R44.S, U$12.3
- new net POWER1: K12.P, X7-2.S
- new net PWM: I/O_PWM.2, K11.1, LED0.C
- new net RA0: U$12.4
- new net RA1: U$12.6
- new net RA2: U$12.11
- new net RC0: U$12.12
- new net RC1: U$12.13
- new net RC2: U$12.14
- new net RD+: R24.1, RL7.1, U$4.D+
- new net RD-: R31.1, RL1.1, U$4.D-
- new net XTAL1: C2.2, R13.1, U$4.XTAL2, X3.P$1
- net +5V: now also C16.1, C19.2, C20.2, C22.1, C23.1, C4.2, I/O_PWM.5, IC2.+V, IC3P.V+, J6.5, J8.5, K11.2, K21.2, R22.1, R30.2, R41.2, R43.2, R44.A, RL0.2, RL9.2, U$12.2, U$9.VDD, X1-1.S
- net +5V/1: now also U$4.AVCC, U$4.AVCC1, U$4.UVCC, U$4.VCC, U$4.VCC1; no longer C17.1, C18.1, C4.1, L_AVCC.1, U$2.VCC, U$2.VCC1, X6-3.S, X6-37.S
- net 3.3V: no longer X6-29.S
- net A0: now also U$4.PF7(ADC7(TDI); no longer U$2.PF7(ADC7)
- net A1: now also R33.1, U$4.PF6(ADC6/TDO); no longer R.1, U$2.PF6(ADC6)
- net A2: now also U$4.PF5(ADC5/TMS); no longer U$2.PF5(ADC5)
- net A3: now also R.1, U$4.PF4(ADC4/TCK); no longer R33.1, U$2.PF4(ADC4)
- net A4: now also U$4.PF1(ADC1); no longer U$2.PF3(ADC3)
- net A5: now also U$4.PF0(ADC0); no longer R35.1, U$2.PF2(ADC2)
- net AREF: now also U$4.AREF; no longer U$2.AREF
- net CS: now also U$4.PD4(ICP1/ADC8); no longer U$2.PD4(ICP1)
- net D10*: now also Q2.G, U$4.PB6(OC1B/OC4B/ADC13); no longer Q4.G, U$2.PB6(OC1B)
- net D11*: now also Q6.G, U$4.PB7(OC0A/OC1C/RTS); no longer Q5.G, U$2.PB7(OC0A/OC1C)
- net D12*: now also C6.1, R9.2, U$4.PD6(T1/ADC9/!OC4D); no longer U$2.PD6(T1)
- net D13*: now also U$4.PC7(ICP3/CLK0/OC4A); no longer U$2.PE3(IUID)
- net D5*: now also Q5.G, U$4.PC6(OC3A/!OC4A); no longer Q6.G, U$2.PE7(INT7/AIN1)
- net D6*: now also Q1.G, U$4.PD7(OC4D/ADC10/T0); no longer U$2.PD7(T0)
- net D7*: now also U$4.PE6(INT.6/AIN0); no longer U$2.PE6(INT6/AIN0)
- net D8*: now also R35.1, U$4.PB4(ADC11); no longer Q1.G, U$2.PB4(OC2A)
- net D9*: now also Q4.G, U$4.PB5(OC1A/ADC12/!OC4B); no longer Q2.G, U$2.PB5(OC1A)
- net GND: now also C14.1, C15.2, C16.2, C17.1, C18.1, C19.1, C20.1, C21.1, C22.2, C23.2, C4.1, I/O_PWM.4, IC2.-V, IC2.REF, IC3P.V-, J6.4, J6.6, J8.4, J8.6, LED13.C, LED14.C, LED16.C, Q3.S, R36.1, R38.1, R42.1, R44.E, U$12.1, U$12.10, U$12.5, U$12.7, U$12.8, U$12.9, U$4.GND, U$4.GND1, U$4.GND2, U$4.GND3, U$4.UGND, U$5.1, U$5.2, U$9.VSS, X1-4.S; no longer C16.1, C17.2, C18.2, C4.2, U$2.GND, U$2.GND1, U$2.GND2, U$2.UGND, X6-39.S
- net HWB: now also U$4.PE2(!HWB); no longer U$2.PE2(HWB)
- net MISO: now also U$4.PB3(PDO/MISO); no longer U$2.PB3(PD0/MISO)
- net MOSI: now also U$4.PB2(PDI/MOSI); no longer U$2.PB2(PD1/MOSI)
- net N$13: now also IC2.RG@1, R2.2; no longer C6.1, L_AVCC.2, U$2.AVCC
- net N$14: now also LED14.A, RL7.2; no longer C2.2, U$2.XTAL1, X3.P$2
- net N$2: now also IC3B.-IN, IC3B.OUT, R26.1, U$2.GND, V1.1
- net N$39: now also IC3A.+IN, U$2.OUT; no longer C8.2, U$2.XTAL2, X3.P$1
- net N$8: now also LED13.A, RL1.2; no longer C3.2, U$2.UCAP
- net RESET: now also U$4./RESET; no longer U$2.RESET
- net RX: now also U$4.PD2(INT2/RXD1); no longer U$2.PD2(INT2/RXD1)
- net RXLED: now also U$4.PB0(SS); no longer U$2.PB0(SS)
- net SCK: now also U$4.PB1(SCK); no longer U$2.PB1(SCLK)
- net SCL: now also J8.2, U$4.PD0(INT0/OC0B/SCL), U$9.SCL; no longer U$2.PD0(INT0/SCL/PD0)
- net SDA: now also J8.3, U$4.PD1(INT1/SDA), U$9.SDA; no longer U$2.PD1(INT1/SDA/OC2B)
- net TX: now also U$4.PD3(INT3/TXD1); no longer U$2.PD3(INT3/TXD1)
- net TXLED: now also U$4.PD5(XCK/CTS); no longer U$2.PD5(XCK1)
- net VUSB: now also U$4.VBUS; no longer C16.2, U$2.UVCC, U$2.VBUS
Other:
- note added: "ATMega32u4"
- note added: "Keypad"
- note added: "LCD"
- note added: "Relay"
- note added: "Weight"
- note added: "pH meter"
- note removed: "AT90usb1286"
- moved on the sheet: C11, C16, C17, C18, C2, C3, C4, C6, C7, C8, C9, I2C-J4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
