File: PCB/IntegratedBertha/v1_1cRouted/integratedBertha.sch (EAGLE design)
At the start: 65 parts, among them CON1 SPI, IC1 REG1117, Q3 BSP75, Q5 BSP75, U1 MPL3115A2LGA8, X3 16MHz, X4 MINI-USB

Commit message: corrected boards to fulfill design rules of the factory in Bogota (drill size and copper spacing. small changes in solardecathlon (SPI pins and design rules changed for zigbee header pads
Parts:
- removed JP1, JP2, JP3, JP4, JP5, JP6: (no value), SparkFun:M02LOCK_LONGPADS
- removed JP10, JP7, JP8, JP9: (no value), SparkFun:M03LONGPADS
- removed JP13: (no value), SparkFun:M04LOCK_LONGPADS
- removed LED3: RED, adafruit:LEDCHIP-LED0805
- removed Q3: BSP75, infineon:BSP613P
- removed U1: MPL3115A2LGA8, SparkFun-Sensors:MPL3115A2LGA8
- added 12V-OK, 3.3V-OK, 5V-OK: RED, adafruit:LEDCHIPLED_1206
- added BLINK: GREEN, adafruit:LEDCHIPLED_1206
- added C16: 100nF, rcl:C-EUC1206
- added D5: 1N581D1206, lpatiny:1N581D1206
- added I/O1, I/O2, I/O3, I/O4, I/O5: RJ12, lpatiny:RJ12STRAIGHT
- added I2C: RJ12STRAIGHT-I2C, lpatiny:RJ12STRAIGHT-I2C
- added IC2: AD8223, analog-devices:AD620R
- added J7: 22--02, lpatiny:22--02
- added L1: 10uH, rcl:L-USL2012C
- added LED2, LED5, LED6, LED8: Blue, adafruit:LEDCHIPLED_1206
- added LED7: BLue, adafruit:LEDCHIPLED_1206
- added Q1, Q2, Q4, Q6: BSP75, infineon:BSP613P
- added Q7: IRF3704S, transistor-power:IRF3704S
- added R, R17, R25, R32, R33, R34, R35: 1k, rcl:R-EU_R0805
- added R10, R21: 4.7k, resistor:R-EU_R1206
- added R16, R18: 10k, rcl:R-EU_R0805
- added R19, R20: 49.9, resistor:R-EU_R1206
- added R28, R29: 10K, resistor:R-EU_M0805
- added RL2, RL3, RL5, RL6, RL8: 1K, rcl:R-EU_R0805
- added RL4: 1K, resistor:R-EU_R0805
- added X1: 22-23-20415.08S, lpatiny:22-23-20415.08S
- added X2, X5: 22-23-20315.08S, lpatiny:22-23-20315.08S
- C13: value 100nF -> 4.7uF
- C14: value 10uF -> 100nF
- C6: value 220nF -> 330nF
- CON1: device lpatiny:TINYISPTAG -> lpatiny:TINYISPT
- LED11, LED12, LED9: device adafruit:LEDCHIP-LED0805 -> adafruit:LEDCHIPLED_1206
- R1: value 4.7k -> 10k; device resistor:R-EU_M1206 -> rcl:R-EU_R0805
- R2: value 10k -> 300; device resistor:R-EU_M1206 -> resistor:R-EU_R1206
- R4, R5, R6, R7: value 4.7k -> 1k; device resistor:R-EU_M1206 -> rcl:R-EU_R0805
- R9: value 10k -> 100; device resistor:R-EU_M1206 -> resistor:R-EU_R1206
- U$1: value M24512 -> SST25VF064C; device lpatiny:M24512 -> BertaLib:SST25VF064C
- U$2: value CHIPCAP -> STARGND; device lpatiny:CHIPCAP -> lpatiny:STARGND
- U$3: value SZ05-ZIGBEETHROUGHHOLE -> SZ05-ZIGBEE
- U$4: value ATMEGA32U4-AU -> ATMEGA32U4
- U$6: value DS1820 -> KPJX-4S-S; device Ava:DS1820 -> lpatiny:KPJX-4S-S
Connections:
- net D+USB renamed USBC_P
- net D-USB renamed USBC_N
- net RD+ renamed USB_P
- net RD- renamed USB_N
- removed net $1: C13.2, C14.2, C15.2, JP3.1, U1.GND
- removed net $12: JP2.1, U$1.VSS
- removed net $2: C4.2, C6.2, JP4.1, U$2.GND
- removed net $3: JP5.1, U$6.GND
- removed net GND_CONTROLLED: JP13.4, JP2.2, JP3.2, JP4.2, JP5.2, Q3.D@1, Q5.S
- removed net N$8: JP6.1, U$3.GND
- removed net VCC: C10.1, C12.2, C5.1, D2.C, D3.C, D4.C, IC1.VIN, R15.2, U$4.AVCC, U$4.AVCC1, U$4.UVCC, U$4.VCC, U$4.VCC1
- new net +12V: I/O1.1, I/O2.1, I/O3.1, I/O4.1, I/O5.1, I2C.1, J7-1.S, RL3.2, U$6.+12V
- new net +5V/1: C10.1, C12.2, C5.1, D2.C, D3.C, D4.C, IC1.VIN, R15.2, RL4.1, U$4.AVCC1, U$4.UVCC, U$4.VCC, U$4.VCC1
- new net AGND: C11.2, C14.1, C15.2, C16.1, C4.1, C6.2, IC2.-V, IC2.REF, U$2.AGND, U$4.GND2, U$4.GND3, X1-4.S
- new net DIFF+: C13.1, C14.2, IC2.+, R19.1
- new net DIFF-: C13.2, C15.1, IC2.-, R20.1
- new net FMOSI: D5.A, R1.1, U$1.MOSI
- new net N$1: I/O3.2, LED6.C, Q4.D@1
- new net N$10: R16.1, R17.1, U$1.CS
- new net N$12: 5V-OK.A, RL4.2
- new net N$14: C16.2, L1.1, U$4.AVCC
- new net N$15: IC2.RG@2, R2.1
- new net N$17: LED2.A, R25.1
- new net N$18: I/O1.3, R.2
- new net N$19: I/O5.2, LED8.C, Q6.D@1
- new net N$21: R10.2, RL6.2, X2-2.S
- new net N$22: LED6.A, R5.1
- new net N$23: R18.2, U$1.SCK
- new net N$28: I/O2.2, LED5.C, Q2.D@1
- new net N$29: I/O4.3, R34.2
- new net N$3: BLINK.A, RL5.2
- new net N$30: LED7.A, R6.1
- new net N$31: R20.2, X1-2.S
- new net N$32: I/O5.3, R35.2
- new net N$33: LED8.A, R7.1
- new net N$34: I/O1.2, LED2.C, Q1.D@1
- new net N$36: J7-2.S, Q7.D
- new net N$37: R19.2, X1-3.S
- new net N$4: LED5.A, R4.1
- new net N$40: IC2.OUT, R9.1
- new net N$5: I/O4.2, LED7.C, Q5.D@1
- new net N$7: I/O3.3, R33.2
- new net N$75: 12V-OK.A, RL3.1
- new net N$9: R21.2, RL8.2, X5-2.S
- net +5V: now also C4.2, I/O1.5, I/O2.5, I/O3.5, I/O4.5, I/O5.5, I2C.5, IC2.+V, L1.2, R10.1, R21.1, R25.2, R28.1, R29.1, R4.2, R5.2, R6.2, R7.2, U$6.+5V, X1-1.S, X2-1.S, X5-1.S; no longer JP1.1
- net 3.3V: now also R1.2, R16.2, U$1.HOLD, U$1.WP; no longer C13.1, C14.1, C6.1, JP10.1, JP13.1, JP7.1, JP8.1, JP9.1, R1.1, R2.2, R4.1, R5.1, R6.1, R7.1, R9.1, U$2.VDD, U$6.VCC, U1.VDD, U1.VDDIO
- net A0: now also RL6.1; no longer R4.2, U$6.DQ
- net A1: now also R33.1; no longer JP9.2, R6.2
- net A2: now also R32.1; no longer JP8.2, R5.2
- net A3: now also R.1; no longer JP7.2, R1.2
- net A4: now also R34.1; no longer JP10.2, R7.2
- net A5: now also RL8.1
- net CS: now also R17.2
- net D10*: now also Q2.G
- net D11*: now also Q6.G
- net D12*: now also C6.1, R9.2
- net D13*: now also RL5.1
- net D5*: now also Q5.G
- net D6*: now also Q1.G; no longer Q5.G
- net D7*: now also RL2.1
- net D8*: now also R35.1; no longer Q3.G
- net D9*: now also Q4.G
- net GND: now also 12V-OK.C, 3.3V-OK.C, 5V-OK.C, BLINK.C, I/O1.4, I/O1.6, I/O2.4, I/O2.6, I/O3.4, I/O3.6, I/O4.4, I/O4.6, I/O5.4, I/O5.6, I2C.4, I2C.6, Q1.S, Q2.S, Q4.S, Q5.S, Q6.S, Q7.S, U$1.GND, U$2.DGND, U$2.GND, U$3.GND, U$6.GND1, U$6.GND2, X2-3.S, X5-3.S; no longer C11.2, JP1.2, JP10.3, JP7.3, JP8.3, JP9.3, LED3.C, Q3.S, U$1.-WC, U$1.E0, U$1.E1, U$1.E2, U$4.GND2, U$4.GND3
- net MISO: now also U$1.MISO
- net MOSI: now also D5.C
- net N$13: now also IC2.RG@1, R2.2; no longer C15.1, U1.CAP
- net N$2: now also I/O2.3, R32.2; no longer JP6.2, Q5.D@1
- net N$20: now also 3.3V-OK.A; no longer LED3.A
- net N$6: now also Q7.G, RL2.2; no longer C4.1, U$2.VCORE
- net SCK: now also R18.1
- net SCL: now also I2C.2, R28.2; no longer JP13.2, R9.2, U$1.SCL, U$2.SCL, U1.SCL
- net SDA: now also I2C.3, R29.2; no longer JP13.3, R2.1, U$1.SDA, U$2.SDA, U1.SDA
Other:
- note added: "Flash Memory"
- note added: "One wire"
- note added: "PID"
- note added: "RJ12"
- note added: "RS232 (Bluetooth) & i2c"
- note added: "Weight"
- note removed: "I2C Memory"
- note removed: "ZigBee"
- moved on the sheet: C13, C14, C15, C4, C6, Q5, R1, R2, R4, R5, R6, R7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
