File: PCB/SolarDecathlon/v1.1/v1.brd (EAGLE design)
At the start: 95.4 x 46.5 mm, 65 parts, among them CON1 SPI, IC1 REG1117, Q3 BSP75, Q5 BSP75, U1 MPL3115A2LGA8, X3 16MHz, X4 MINI-USB

Commit message: corrected boards to fulfill design rules of the factory in Bogota (drill size and copper spacing. small changes in solardecathlon (SPI pins and design rules changed for zigbee header pads
Parts:
- CON1: device lpatiny:TC2030-MCP -> lpatiny:TC2030-MCP-NL
- moved U$3 0.05 mm to (83.9, 14.6)
Routing:
- net MOSI: track 27.6 -> 109.5 mm, vias 5 -> 3
- net VCC: track 156.0 -> 115.9 mm, vias 9 -> 4
- net SCL: track 100.3 -> 137.7 mm
- net N$2: track 45.4 -> 77.9 mm, vias 2 -> 0
- net SCK: track 55.2 -> 87.4 mm
- net 3.3V: track 215.7 -> 186.8 mm, vias 6 -> 3
- net D6*: track 27.2 -> 55.4 mm
- net A3: track 91.3 -> 69.6 mm, vias 1 -> 2
- net ISP+5V: track 53.2 -> 33.8 mm, vias 0 -> 2
- net RESET: track 76.7 -> 61.5 mm, vias 2 -> 4
- net MISO: track 61.4 -> 47.1 mm
- net SDA: track 90.1 -> 103.3 mm
- net +5V: track 109.5 -> 96.9 mm
- net D-USB: track 19.8 -> 7.84 mm
- net GND: track 392.5 -> 383.3 mm, vias 7 -> 4
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- added copper zone on layer 16, net GND
Other:
- board text removed: "w5100"
