File: PCB/SolarDecathlon/v1.1/v1.sch (EAGLE design)
At the start: 65 parts, among them CON1 SPI, IC1 REG1117, Q3 BSP75, Q5 BSP75, U1 MPL3115A2LGA8, X3 16MHz, X4 MINI-USB

Commit message: corrected boards to fulfill design rules of the factory in Bogota (drill size and copper spacing. small changes in solardecathlon (SPI pins and design rules changed for zigbee header pads
Parts:
- CON1: device lpatiny:TINYISPTAG -> lpatiny:TINYISPT
